File: hardware/schematics/esc/esc_main.kicad_sch (KiCad schematic)
At the start: 53 parts, among them J1 SM08B-SRSS-TB, U1 TLV76733DRVR, U12 INA186A3IDCKR, U18 LMR51420YDDCR, U5 XRIM160808SR47MBCD

Commit message: Refresh design sources: import rev2 sheets + libs from current sibling repos
FC sheets   <- OpenFC-Lite-Mini rev2 (RP2354A, LMR51430 power tree, COS8051 OSD)
ESC sheets  <- 4in1-mini Rev2 (AT32F421 + NSG2065Q + DOY180N03T, INA186 CSA)
ELRS sheet  <- OpenRX-Lite (ESP32-C3 + SX1281, chip antenna)

Drop-in swaps at paths the root sheet already references; esc_channel
instantiated 4x from root resolves. esc_main.kicad_sch (4in1-mini top:
buck/LDO/CSA/TVS/connector) kept as reference, with ESC.kicad_sch beside
it so its internal channel instances resolve if ever instantiated.

Libraries replaced wholesale: lib(.kicad_sym/.pretty/.3dshapes) from
OpenFC-Lite-Mini, components+4in1ESC from 4in1-mini, OpenRX-Shared from
OpenRX. 3D model paths in OpenRX-Shared.pretty rewritten to project-
local via pcbnew API. Hierarchy verified with kicad-cli netlist export.

Supersedes the 2026-04 port from OpenFC-ECO V0.3 / 4in1ESC 2 (in git
history). Schematic re-annotation + root rewiring is manual work in
KiCad. Old PCB layout retained; footprints are embedded so it opens,
but layout predates this refresh.

Co-Authored-By: Claude Fable 5 <noreply@anthropic.com>
Parts:
- removed C10, C11, C12, C13, C14, C15, C16, C17, C18, C19, C2, C20, C21, C22, C23, C24, C25, C26, C27, C28, C29, C3, C31, C4, C40, C41, C47, C5, C51, C6, C7, C8, C9: 10uF, Capacitor_SMD:C_0805_2012Metric, symbol Device:C
- removed U18: LMR51420YDDCR, lib:SOT-23-6_L2.9-W1.6-P0.95-LS2.9-BL, symbol lib:LMR51420YDDCR_ESC
- added CL32: 10uF, Capacitor_SMD:C_1206_3216Metric, symbol Device:C
- added D1, D2: SMF24A-T13, 4in1ESC:SOD-123FL_L2.7-W1.8-LS3.7-RD, symbol components:SMF24A-T13
- added U13: LMR54406DBVR, 4in1ESC:SOT-23-6_L2.9-W1.6-P0.95-LS2.8-BR, symbol components:LMR54406DBVR
- C1, C42: Cost (none) -> 0.037; MPN (none) -> CL05A226MQ5QUNC
- C43, C86: Cost (none) -> 0.04157; MPN (none) -> CL10A226MO7JZNC
- C69, C70, C71, C72, C93, C94: symbol lib:GRM033R61C104KE84D -> ESCLibrary:GRM033R61C104KE84D; Cost (none) -> 0.008457; MPN (none) -> GRM033R6YA104KE14D
- J1: footprint lib:JST_SM08B-SRSS-TB -> 4in1ESC:JST_SM08B-SRSS-TB; symbol lib:SM08B-SRSS-TB -> components:SM08B-SRSS-TB; Cost (none) -> 0.2523; MPN (none) -> SM08B-SRSS-TB(LF)(SN)
- R118: footprint Capacitor_SMD:C_0201_0603Metric -> 4in1ESC:R_0201_0603Metric; Cost (none) -> 0.0007714; MPN (none) -> RC0201FR-0710KL
- R119: value 124k -> 115k; Cost (none) -> 0.0005429; LCSC C423759 -> C166378; MPN (none) -> RTT011153FTH
- R73: footprint Capacitor_SMD:C_0201_0603Metric -> 4in1ESC:R_0201_0603Metric; symbol lib:0201_1kR -> ESCLibrary:0201_1kR; Cost (none) -> 0.0006; MPN (none) -> 0201WMF1001TEE
- Rsense1: Cost (none) -> 0.2657; MPN (none) -> ASR-S-3-0.2F
- U1: footprint lib:WSON-6_L2.0-W2.0-P0.65-TL-EP -> 4in1ESC:WSON-6_L2.0-W2.0-P0.65-TL-EP; symbol lib:TLV76733DRVR -> components:TLV76733DRVR; Cost (none) -> 0.242; MPN (none) -> TLV76733DRVR; Manufacturer (none) -> Texas Instruments
- U12: footprint lib:SOT-363_SC-70-6 -> 4in1ESC:SOT-363_SC-70-6; symbol lib:INA186A3IDCKR -> components:INA186A3IDCKR; Cost (none) -> 0.79; MPN (none) -> INA186A3IDCKR; Manufacturer (none) -> Texas Instruments
- U4: footprint lib:4in1ESC -> 4in1ESC:4in1ESC; symbol lib:4in1ESC -> components:4in1ESC
- U5: value XRIM160808SR47MBCD -> FTC160808S4R7MBCA; footprint lib:IND-SMD_L1.6-W0.8_FTC160865SR47MBCA -> 4in1ESC:IND-SMD_L1.6-W0.8_FTC160865SR47MBCA; symbol lib:XRIM160808SR47MBCD -> components:XRIM160808SR47MBCD; Cost (none) -> 0.1079; LCSC C48391583 -> C46594347; MPN (none) -> FTC160808S4R7MBCA
Connections:
- net +BATT: now also CL32.1, D1.1 (K), D2.1 (K), U13.4 (EN), U13.5 (VIN)
- net GND: now also CL32.2, D1.2 (A), D2.2 (A), U13.2 (GND)
- net at R118.1, R119.2: now also U13.3 (FB)
- net at C72.1, U5.1: now also U13.6 (SW)
- net at C72.2: now also U13.1 (CB)
- net +8V renamed +10V
Other:
- note added: "06/06/2026"
- note added: "2"
- note added: "4 to 36V, can handle 50V spikes. TBD on 8S 1.1Mhz, 0.6A (plenty for gate driving)"
- note added: "No telemetry signal pin, handled by Extended DSHOT protocol"
- note added: "Overview of OpenESC"
- note added: "SMFJ24A means there will be some leakage at fully charged 6S (25.2V) but voltage clamping gets improved too, will monitor this tradeoff"
- note added: "Total array of 20 decoupling caps At 25V DC Bias, only 1.5uF - 2uF derated per cap, so 30 - 40uF but very low ESR"
- moved on the sheet: C1, C42, C43, C69, C70, C71, C72, C86, R118, R119, U1
