File: hardware/schematics/fc/osd.kicad_sch (KiCad schematic)
At the start: 17 parts, among them U22 SN74LVC1G3157DTBR, U23 TLV9061IDPWR, U24 TLV3201AIDBVR

Commit message: Refresh design sources: import rev2 sheets + libs from current sibling repos
FC sheets   <- OpenFC-Lite-Mini rev2 (RP2354A, LMR51430 power tree, COS8051 OSD)
ESC sheets  <- 4in1-mini Rev2 (AT32F421 + NSG2065Q + DOY180N03T, INA186 CSA)
ELRS sheet  <- OpenRX-Lite (ESP32-C3 + SX1281, chip antenna)

Drop-in swaps at paths the root sheet already references; esc_channel
instantiated 4x from root resolves. esc_main.kicad_sch (4in1-mini top:
buck/LDO/CSA/TVS/connector) kept as reference, with ESC.kicad_sch beside
it so its internal channel instances resolve if ever instantiated.

Libraries replaced wholesale: lib(.kicad_sym/.pretty/.3dshapes) from
OpenFC-Lite-Mini, components+4in1ESC from 4in1-mini, OpenRX-Shared from
OpenRX. 3D model paths in OpenRX-Shared.pretty rewritten to project-
local via pcbnew API. Hierarchy verified with kicad-cli netlist export.

Supersedes the 2026-04 port from OpenFC-ECO V0.3 / 4in1ESC 2 (in git
history). Schematic re-annotation + root rewiring is manual work in
KiCad. Old PCB layout retained; footprints are embedded so it opens,
but layout predates this refresh.

Co-Authored-By: Claude Fable 5 <noreply@anthropic.com>
Parts:
- removed R118, R119: 470R, Resistor_SMD:R_0201_0603Metric, symbol Device:R
- removed U23: TLV9061IDPWR, lib:X2SON-4_L0.8-W0.8-P0.48-TL-DPW, symbol lib:TLV9061IDPWR
- removed U24: TLV3201AIDBVR, lib:SOT-23-5_L3.0-W1.7-P0.95-LS2.8-BR, symbol lib:TLV3201AIDBVR
- added R46, R47: 510R, Resistor_SMD:R_0201_0603Metric, symbol Device:R
- added U1: COS8051SOT, lib:SOT-23-5_L3.0-W1.7-P0.95-LS2.8-BR, symbol lib:COS8051SOT
- added U2: TLV7031DPWR, lib:X2SON-4_L0.8-W0.8-P0.48-TL-A, symbol lib:TLV7031DPWR
- D9: renamed from D10; LCSC (none) -> C151629; LCSC Part C151629 -> (none)
- U18: renamed from U22; LCSC (none) -> C2673087; LCSC Part C2673087 -> (none)
- renumbered C106 to C38, C107 to C39, C108 to C40, C109 to C41, C110 to C42, R113 to R41, R114 to R42, R115 to R43, R116 to R44, R117 to R45, R120 to R48
Connections:
- net +3.3V: now also U1.5 (+VS), U2.2 (VCC)
- net GND: now also R46.2, U1.2 (-VS), U2.3 (IN-), U2.5 (VEE)
- net OSD_SYNC: now also U2.1 (OUT)
- net VID_DC: now also U2.4 (IN+)
- net at R48.1: now also R47.2, U1.1 (OUT)
- net at U18.4 (A): now also U1.3 (IN+)
- new net: R46.1, R47.1, U1.4 (IN-)
Other:
- note added: "06/06/2026"
- note added: "2"
- note added: "75R input terminatiom"
- note added: "Analog OSD using PIO State Machine on RP2350"
- note added: "Comparator detects sync pulses, read by RP2350 PIO"
- note added: "Resistor divider let's GPIO port select between high (VOH = 1V: white) or low (VOL = 0.3v: black)"
- moved on the sheet: R48
