File: hardware/schematics/fc/pads.kicad_sch (KiCad schematic)
At the start: 40 parts, among them J1 5V, J10 5V, J11 5V, J12 5V, J13 5V, J14 5V, J15 5V, J16 5V, J17 5V, J18 5V, J19 5V, J2 5V, J20 5V, J21 5V, J22 5V, J23 5V, J24 5V, J25 5V, J26 5V, J27 5V, J28 5V, J29 5V, J3 5V, J30 5V, J31 5V, J32 5V, J33 5V, J34 5V, J35 5V, J36 5V, J37 5V, J38 5V, J39 5V, J4 5V, J5 5V, J6 5V, J7 5V, J8 5V, J9 5V, U12 SM06B-SRSS-TB(LF)(SN)

Commit message: Refresh design sources: import rev2 sheets + libs from current sibling repos
FC sheets   <- OpenFC-Lite-Mini rev2 (RP2354A, LMR51430 power tree, COS8051 OSD)
ESC sheets  <- 4in1-mini Rev2 (AT32F421 + NSG2065Q + DOY180N03T, INA186 CSA)
ELRS sheet  <- OpenRX-Lite (ESP32-C3 + SX1281, chip antenna)

Drop-in swaps at paths the root sheet already references; esc_channel
instantiated 4x from root resolves. esc_main.kicad_sch (4in1-mini top:
buck/LDO/CSA/TVS/connector) kept as reference, with ESC.kicad_sch beside
it so its internal channel instances resolve if ever instantiated.

Libraries replaced wholesale: lib(.kicad_sym/.pretty/.3dshapes) from
OpenFC-Lite-Mini, components+4in1ESC from 4in1-mini, OpenRX-Shared from
OpenRX. 3D model paths in OpenRX-Shared.pretty rewritten to project-
local via pcbnew API. Hierarchy verified with kicad-cli netlist export.

Supersedes the 2026-04 port from OpenFC-ECO V0.3 / 4in1ESC 2 (in git
history). Schematic re-annotation + root rewiring is manual work in
KiCad. Old PCB layout retained; footprints are embedded so it opens,
but layout predates this refresh.

Co-Authored-By: Claude Fable 5 <noreply@anthropic.com>
Parts:
- added J1, J11, J12, J13, J14, J2, J29, J31, J33, J35, J37, J39, J41, J5, J8: 5V, lib:small_pad, symbol Connector_Generic:Conn_01x01
- added P1: SM08B-SRSS-TB(LF)(SN), lib:CONN-TH_SM08B-SRSS-TB-LF-SN, symbol lib:SM08B-SRSS-TB(LF)(SN)
- J17: renamed from J9; now fitted; now in the parts list
- J20: renamed from J12; now fitted; now in the parts list
- J24: renamed from J16; now fitted; now in the parts list
- J36: renamed from J24; now not fitted
- J38: renamed from J25; now not fitted
- J4: renamed from J2; now not fitted
- J47: renamed from J32; now not fitted
- J50: renamed from J35; now not fitted
- J52: renamed from J37; now not fitted
- J53: renamed from J38; now not fitted
- J54: renamed from J39; now not fitted
- J7: renamed from J4; now not fitted
- U8: renamed from U12; LCSC (none) -> C160405; LCSC Part C160405 -> (none)
- renumbered J6 to J10, J7 to J15, J8 to J16, J10 to J18, J11 to J19, J13 to J21, J14 to J22, J15 to J23, J17 to J25, J18 to J26, J19 to J27, J20 to J28, J1 to J3, J21 to J30, J22 to J32, J23 to J34, J26 to J40, J27 to J42, J28 to J43, J29 to J44, J30 to J45, J31 to J46, J33 to J48, J34 to J49, J36 to J51, J3 to J6, J5 to J9
Connections:
- net +5V: now also J5.1 (Pin_1)
- net GND: now also J1.1 (Pin_1), J13.1 (Pin_1), J14.1 (Pin_1), J31.1 (Pin_1), P1.10, P1.2, P1.9
- net PIOUART0_RX: now also P1.4
- net DIGITAL_RX renamed UART0_RX
- net DIGITAL_TX renamed UART0_TX
- net I2C_SCL renamed I2C0.SCL
- net I2C_SDA renamed I2C0.SDA
- net SBUS renamed UART1_RX
- net UART1_RX: now also J8.1 (Pin_1)
- new net +BATT: J29.1 (Pin_1), P1.1
- new net ADC2: J11.1 (Pin_1)
- new net CURRENT: J33.1 (Pin_1), P1.3
- new net M1: J35.1 (Pin_1), P1.5
- new net M2: J37.1 (Pin_1), P1.6
- new net M3: J39.1 (Pin_1), P1.7
- new net M4: J41.1 (Pin_1), P1.8
- new net RSSI: J2.1 (Pin_1)
- new net UART1_TX: J12.1 (Pin_1)
Other:
- note added: "06/06/2026"
- note added: "2"
- note added: "20x20 has 1 less uart, no external ADC's, only 2 LED pads"
- note added: "Camera + VTX"
- note added: "ESC"
- note added: "EXTRA ADC"
- note added: "I2C out"
- note added: "RSSI"
- note added: "RX pads"
- note added: "Solder pads and JST connectors for I/O"
- note removed: "i2C out"
- moved on the sheet: J45, J46, J48, J49, J51
