File: hardware/schematics/fc/rp2350a.kicad_sch (KiCad schematic)
At the start: 53 parts, among them Q1 DMN1150UFB-7B, Q2 DMN1150UFB-7B, Q3 DMN1150UFB-7B, U2 TS2306A 240GF MSM 9_C2976675, U3 RP2354B_C39843328, X1 XTM25012000JT00351001

Commit message: Refresh design sources: import rev2 sheets + libs from current sibling repos
FC sheets   <- OpenFC-Lite-Mini rev2 (RP2354A, LMR51430 power tree, COS8051 OSD)
ESC sheets  <- 4in1-mini Rev2 (AT32F421 + NSG2065Q + DOY180N03T, INA186 CSA)
ELRS sheet  <- OpenRX-Lite (ESP32-C3 + SX1281, chip antenna)

Drop-in swaps at paths the root sheet already references; esc_channel
instantiated 4x from root resolves. esc_main.kicad_sch (4in1-mini top:
buck/LDO/CSA/TVS/connector) kept as reference, with ESC.kicad_sch beside
it so its internal channel instances resolve if ever instantiated.

Libraries replaced wholesale: lib(.kicad_sym/.pretty/.3dshapes) from
OpenFC-Lite-Mini, components+4in1ESC from 4in1-mini, OpenRX-Shared from
OpenRX. 3D model paths in OpenRX-Shared.pretty rewritten to project-
local via pcbnew API. Hierarchy verified with kicad-cli netlist export.

Supersedes the 2026-04 port from OpenFC-ECO V0.3 / 4in1ESC 2 (in git
history). Schematic re-annotation + root rewiring is manual work in
KiCad. Old PCB layout retained; footprints are embedded so it opens,
but layout predates this refresh.

Co-Authored-By: Claude Fable 5 <noreply@anthropic.com>
Parts:
- removed C25, C38, C40, C43: 100n, Capacitor_SMD:C_0201_0603Metric, symbol Device:C
- removed C39, C41, C42: 4.7uF, Capacitor_SMD:C_0402_1005Metric, symbol Device:C
- removed D1: USBLC6-2P6, Package_TO_SOT_SMD:SOT-666, symbol lib:USBLC6-2SC6
- removed L1: AOTA-B201610S3R3-101-T, lib:IND-SMD_L2.0-W1.6_AOTA-B201610S3R3-101-T, symbol lib:AOTA-B201610S3R3-101-T
- removed Q1, Q2, Q3: DMN1150UFB-7B, lib:DFN-3L_L1.0-W0.6-P0.65-BR, symbol lib:DMN1150UFB-7B
- removed R10, R14, R23: 10k, Resistor_SMD:R_0201_0603Metric, symbol Device:R
- removed R11, R12, R13: 30R, Resistor_SMD:R_0201_0603Metric, symbol Device:R
- removed R16, R17, R21: 2.2k, Resistor_SMD:R_0201_0603Metric, symbol Device:R
- removed R18, R19: 1k, Resistor_SMD:R_0201_0603Metric, symbol Device:R
- removed R20: 100k, Resistor_SMD:R_0201_0603Metric, symbol Device:R
- removed R25, R8: 200R, Resistor_SMD:R_0201_0603Metric, symbol Device:R
- removed U2: TS2306A 240GF MSM 9_C2976675, lib:SW-SMD_4P-L3.0-W2.0-P0.85-LS3.5, symbol lib:TS2306A240GFMSM9_C2976675
- removed U3: RP2354B_C39843328, lib:QFN-80_L10.0-W10.0-P0.40-TL-EP3.4, symbol lib:RP2354B_C39843328
- added C22: 100n, Capacitor_SMD:C_0201_0603Metric, symbol Device:C
- added C37, C45, C46: 4.7uF, Capacitor_SMD:C_0402_1005Metric, symbol Device:C
- added L4: AOTA-B201610S3R3-101-T, lib:IND-SMD_L2.0-W1.6_AOTA-B201610S3R3-101-T, symbol lib:AOTA-B201610S3R3-101-T
- added Q5, Q6: AP1606, lib:DFN-3L_L1.0-W0.6-P0.65-BR, symbol lib:DMN1150UFB-7B
- added R37: 30R, Resistor_SMD:R_0201_0603Metric, symbol Device:R
- added R38: 10k, Resistor_SMD:R_0201_0603Metric, symbol Device:R
- added R51: 2.4k, Resistor_SMD:R_0201_0603Metric, symbol Device:R
- added R52, R53: 75R, Resistor_SMD:R_0201_0603Metric, symbol Device:R
- added R6, R7: 5.1k, Resistor_SMD:R_0201_0603Metric, symbol Device:R
- added U10: RP2354A, lib:QFN-60_L7.0-W7.0-P0.40-TL-EP3.4, symbol lib:RP2354A
- added U11: TS2306A 240GF MSM 9_C2976675, lib:SW-SMD_4P-L3.0-W2.0-P0.85-LS3.5, symbol lib:TS2306A240GFMSM9_C2976675
- D2: value LED_1_Green -> LED_1_Blue; footprint LED_SMD:LED_0201_0603Metric -> LED_SMD:LED_0402_1005Metric; LCSC C3646922 -> C22355736; MPN XL-0201UGC -> XL-1005UBC
- R24: value 2.2k -> 30R; LCSC C142018 -> C778391; MPN RC0201FR-072K2L -> NQ01WMJ0300TEE; Manufacturer YAGEO -> UNI-ROYAL
- R9: value 10k -> 1k; LCSC C106225 -> C270365; MPN RC0201FR-0710KL -> 0201WMF1001TEE; Manufacturer YAGEO -> UNI-ROYAL
- USB1: LCSC (none) -> C5187472; LCSC Part C5187472 -> (none)
- X1: LCSC (none) -> C37635340; LCSC Part C37635340 -> (none)
- renumbered C24 to C1, C33 to C10, C34 to C11, C35 to C12, C36 to C13, C26 to C3, C27 to C4, C28 to C5, C29 to C6, C30 to C7, C31 to C8, C32 to C9, R2 to R1, R3 to R2, R22 to R23, R4 to R3, R5 to R4, R6 to R5
Connections:
- net D+_C is gone; now on net D+: USB1.A6 (DP1), USB1.B6 (DP2)
- net D-_C is gone; now on net D-: USB1.A7 (DN1), USB1.B7 (DN2)
- net +1.1V: now also C37.1, C46.1, L4.1, U10.23 (DVDD), U10.39 (DVDD), U10.50 (VREG_FB), U10.6 (DVDD)
- net +3.3V: now also R15.1, C45.1, R6.1, R7.1, U10.1 (IOVDD), U10.11 (IOVDD), U10.20 (IOVDD), U10.26 (RUN), U10.30 (IOVDD), U10.38 (IOVDD), U10.44 (ADC_AVDD), U10.45 (IOVDD), U10.49 (VREG_VIN), U10.53 (USB_OTP_VDD), U10.54 (QSPI_IOVDD); no longer R9.1
- net +5V: now also R51.1; no longer R24.1
- net +BATT: now also R1.2; no longer R1.1
- net 10V_ENABLE: now also U10.41 (GPIO27_ADC1)
- net ADC_VBAT: now also R1.1, U10.43 (GPIO29_ADC3); no longer R1.2
- net BEEPER: now also R23.2, Q5.1 (G), U10.28 (GPIO17)
- net BUZZER-: now also Q5.3 (D)
- net D+: now also R37.2
- net D-: now also R24.1
- net ESC_CURRENT: now also R9.1
- net FLASH_CS: now also U10.33 (GPIO21)
- net GND: now also C22.2, C37.2, C45.2, C46.2, Q5.2 (S), Q6.2 (S), U10.47 (VREG_PGND), U10.61 (EP), U11.1
- net GYRO_CS: now also U10.17 (GPIO13)
- net GYRO_INT: now also U10.13 (GPIO9)
- net LED0: now also R52.1, U10.40 (GPIO26_ADC0); no longer R15.1
- net LED_STRIP: now also Q6.3 (D), R51.2
- net LED_STRIP_L: now also Q6.1 (G), U10.12 (GPIO8)
- net MOTOR1: now also U10.37 (GPIO25)
- net MOTOR2: now also U10.36 (GPIO24)
- net MOTOR3: now also U10.35 (GPIO23)
- net MOTOR4: now also U10.34 (GPIO22)
- net OSD_EN: now also U10.19 (GPIO15)
- net OSD_SYNC: now also U10.27 (GPIO16)
- net OSD_W: now also U10.18 (GPIO14)
- net PIOUART0_RX: now also U10.5 (GPIO3)
- net PIOUART0_TX: now also U10.4 (GPIO2)
- net SPI0.MISO: now also U10.32 (GPIO20)
- net SPI0.MOSI: now also U10.31 (GPIO19)
- net SPI0.SCK: now also U10.29 (GPIO18)
- net SPI1.MISO: now also U10.16 (GPIO12)
- net SPI1.MOSI: now also U10.15 (GPIO11)
- net SPI1.SCK: now also U10.14 (GPIO10)
- net UART0_RX: now also U10.3 (GPIO1)
- net UART0_TX: now also U10.2 (GPIO0)
- net UART1_RX: now also U10.10 (GPIO7)
- net UART1_TX: now also U10.9 (GPIO6)
- net XIN: now also U10.21 (XIN)
- net XOUT: now also U10.22 (XOUT)
- net at R24.2: now also U10.51 (USB_DM)
- net at C44.1: now also R15.2, U10.46 (VREG_AVDD)
- net at D2.2 (A): now also R53.2; no longer R15.2
- net ESC_CURR: now reaches R9.2
- net ESC_CURR: now also C22.1, U10.42 (GPIO28_ADC2)
- new net: R38.1, U11.2
- new net: R38.2, U10.60 (QSPI_SS)
- new net: R52.2, R53.1
- new net: L4.2, U10.48 (VREG_LX)
- new net: R37.1, U10.52 (USB_DP)
- new net I2C0.SCL: R6.2, U10.8 (GPIO5)
- new net I2C0.SDA: R7.2, U10.7 (GPIO4)
- no-connect marks 19 -> 9
Other:
- note added: "06/06/2026"
- note added: "2"
- note added: "RP2350 1.1V DC-DC SMPS Follow datasheet guidance on component placement"
- note added: "RP2350 Pin mapping and universal peripherals"
- note added: "RP2354A: Smaller variant with integrated flash (2MB)"
- note added: "USB port"
- note added: "decoupling caps, place close to IC, one is enough when 2 pins are next to each other"
- note added: "gyro SPI"
- note added: "i2c for external sensors"
- note added: "vbat sense. 1/11 scale"
- note removed: "1.1V SMPS by RP datasheet inductor polarity important"
- note removed: "RC lowpass filters on ADC and VREG like Pico datasheet"
- note removed: "RP2350 1.8V DC-DC SMPS Follow datasheet guidance on component placement"
- note removed: "RP2354B: Larger variant with integrated flash (2MB) and more GPIO"
- note removed: "SBUS inverter"
- note removed: "USB port with ESD protection"
- note removed: "decoupling caps, place close to IC"
- note removed: "for external (extra)"
- note removed: "gyro SPI line, seperate from blackbox"
- note removed: "i2c for barometer and external sensors possibly"
- note removed: "vbat sense. 1/10 scale"
- moved on the sheet: C1, C10, C11, C12, C13, C3, C4, C5, C6, C7, C8, C9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
