File: hardware/ESC.kicad_sch (KiCad schematic)
At the start: 36 parts, among them Q1 DOY180N03T, Q2 DOY180N03T, Q3 DOY180N03T, Q4 DOY180N03T, Q5 DOY180N03T, Q6 DOY180N03T, U2 AT32F421G8U7, U3 NSG2065Q

Commit message: Root sheet: place the sub-sheets; ESC as the 4in1 top sheet
esc_4in1.kicad_sch is OpenESC-20x20's 4in1-mini top sheet (battery input,
shunt and INA186 current sense, 12V/3V3 regulators, four ESC channel
instances). Its channel sub-sheet keeps its original file name ESC.kicad_sch
so the top sheet is untouched. Root sheet: Power, IMU, OSD, Blackbox, Pads,
RP2354A, ESC, RX placed, no wiring.
Parts:
- renumbered C32 to C35, C36 to C39, C48 to C78, C49 to C79, C50 to C80, C53 to C83, C57 to C88, Q1 to Q19, Q2 to Q20, Q3 to Q21, Q4 to Q22, Q5 to Q23, Q6 to Q24, R16 to R55, R17 to R56, R18 to R57, R19 to R58, R20 to R59, R21 to R60, R22 to R61, R23 to R62, R24 to R63, R25 to R64, R26 to R65, R27 to R66, R28 to R67, R29 to R68, R30 to R69, R31 to R70, R32 to R71, R33 to R72, R74 to R77, TP1 to TP7, TP4 to TP8, U2 to U10, U3 to U11
