File: hardware/esc_channel.kicad_sch (KiCad schematic)
At the start: 36 parts, among them Q19 DOY180N03T, Q20 DOY180N03T, Q21 DOY180N03T, Q22 DOY180N03T, Q23 DOY180N03T, Q24 DOY180N03T, U10 AT32F421G8U7, U11 NSG2065Q

Commit message: Net classes: VBAT, Phase, Power, Gate, USB, RF, Analog with colours and patterns
Replaces the stale 50Ohm /ELRS/* patterns inherited from the template.
Widths and clearances start from the line standard (0.09/0.09, via 0.35/0.20)
and the ESC boards' practice; USB and RF geometry still to be checked against
the chosen JLCPCB 6-layer stackup.
Parts:
- renumbered C80 to C37, C78 to C38, C79 to C39, C83 to C40, C35 to C41, C39 to C42, C88 to C43, Q19 to Q3, Q20 to Q4, Q21 to Q5, Q22 to Q6, Q23 to Q7, Q24 to Q8, R55 to R35, R56 to R36, R57 to R37, R58 to R38, R59 to R39, R77 to R40, R60 to R41, R61 to R42, R62 to R43, R63 to R44, R64 to R45, R65 to R46, R66 to R47, R67 to R48, R68 to R49, R69 to R50, R70 to R51, R71 to R52, R72 to R53, TP7 to TP1, TP8 to TP2, U10 to U13, U11 to U14

Commit message: OpenAIO: master PCB with Base and Core islands routed, AIO_outline footprint+symbol in project lib
Save point before the two-board (LGA) split tooling.
Parts:
- added C90, C91, C92: C, Capacitor_SMD:C_0805_2012Metric, symbol Device:C
- C37, C38, C39, C40, C41, C42, C43, R35, R36, R37, R38, R39, R40, R41, R42, R43, R44, R45, R46, R47, R48, R49, R50, R51, R52, R53: KiLib_Generator (none) -> SMD_2terminal_chip_molded
Connections:
- net +BATT: now also C90.1, C91.1, C92.1
- net GND: now also C90.2, C91.2, C92.2
