File: hardware/esc_channel.kicad_sch (KiCad schematic)
At the start: 39 parts, among them Q3 DOY180N03T, Q4 DOY180N03T, Q5 DOY180N03T, Q6 DOY180N03T, Q7 DOY180N03T, Q8 DOY180N03T, U13 AT32F421G8U7, U14 NSG2065Q

Commit message: chore: consolidate OpenAIO design assets and guidance
Parts:
- renumbered C37 to C43, C38 to C44, C39 to C45, C40 to C46, C41 to C47, C42 to C48, C43 to C49, C90 to C50, C91 to C51, C92 to C52, Q3 to Q1, Q4 to Q2, Q5 to Q3, Q6 to Q4, Q7 to Q5, Q8 to Q6, R35 to R17, R36 to R18, R37 to R19, R38 to R20, R39 to R21, R40 to R22, R41 to R23, R42 to R24, R43 to R25, R44 to R26, R45 to R27, R46 to R28, R47 to R29, R48 to R30, R49 to R31, R50 to R32, R51 to R33, R52 to R34, R53 to R35, TP1 to TP3, TP2 to TP4, U13 to U11, U14 to U12
