File: hardware/esc_channel.kicad_sch (KiCad schematic)
At the start: 39 parts, among them Q19 DOY180N03T, Q20 DOY180N03T, Q21 DOY180N03T, Q22 DOY180N03T, Q23 DOY180N03T, Q24 DOY180N03T, U10 AT32F421G8U7, U11 NSG2065Q

Commit message: One board: merge Base and Core onto the OpenAIO-Whoop 8L HDI stackup
- hardware/OpenAIO.kicad_pcb: the routed Base and Core layouts of 8fa8d7b
  side by side in one board, all routing kept (Core promoted to 8 layers
  before the append so no Base layer was dropped). J90/J91 LGA deleted;
  their 46 nets are now direct links (51 unconnected, listed in
  research/ROUTING.md). Stackup and board setup from OpenAIO-Whoop:
  8L HDI 1+6+1, 0.997 mm, 1 oz all layers, microvia 0.25/0.10,
  buried 0.33/0.15. Base DRC severities and exclusions kept.
- hardware/OpenAIO.kicad_dru: canonical block, Whoop HDI via rules,
  Base/Core rules that still apply; LGA, 2 oz and 1.6 mm via rules gone.
- Schematic: core_interface sheet removed; DPS368 baro U28 on I2C0;
  review fixes (U3 HF cap C116, RP2354 caps C117/C118, buzzer flyback D10,
  SD card on +3.3V, D9 on +4v5, FLASH_CS -> SD_CS, PWR_FLAGs, U7 pin
  names, ESC cap pin types, L4 LCSC). ERC 32 -> 0 errors.
- Libraries project-local: every footprint, 3D model and symbol in lib;
  OPENDRONE_LIB aliases removed from the lib tables.
- Two-board projects, multiboard config and LGA tools removed; Whoop
  board tools added in hardware/tools.
- Docs: README, AGENTS.md, research/ROUTING.md (hand-over),
  SCHEMATIC-REVIEW-2026-10-15.md, Betaflight target baro.

DRC: 38 errors (25 dangling LGA escape vias, 13 Core leftovers listed),
51 unconnected (the Base-Core links), 0 net or value parity issues.

Co-Authored-By: Claude Opus 5.5 <noreply@anthropic.com>
Parts:
- C35, C39, C83: footprint Capacitor_SMD:C_0402_WIDE -> lib:C_0402_WIDE; symbol ESCLibrary:GRM033R61C104KE84D -> lib:GRM033R61C104KE84D
- C78, C79, C80, C88: footprint Capacitor_SMD:C_0201_0603Metric -> lib:C_0201_0603Metric; symbol ESCLibrary:GRM033R61C104KE84D -> lib:GRM033R61C104KE84D
- C96, C97, C98: footprint Capacitor_SMD:C_0805_2012Metric -> lib:C_0805_2012Metric
- Q19, Q20, Q21, Q22, Q23, Q24: symbol PCM_Transistor_MOSFET_AKL:2N6660 -> lib:2N6660
- R55, R56, R60, R61, R62, R63: footprint Resistor_SMD:R_0201_0603Metric -> lib:R_0201_0603Metric; symbol PCM_Resistor_AKL:R_0402 -> lib:R_0402
- R57, R58, R64, R66, R67, R69, R70, R72: footprint Resistor_SMD:R_0201_0603Metric -> lib:R_0201_0603Metric; symbol ESCLibrary:0201_10kR -> lib:0201_10kR
- R59: footprint Resistor_SMD:R_0201_0603Metric -> lib:R_0201_0603Metric; symbol ESCLibrary:0201_220R -> lib:0201_220R
- R65, R68, R71: footprint Resistor_SMD:R_0201_0603Metric -> lib:R_0201_0603Metric; symbol ESCLibrary:0201_1kR -> lib:0201_1kR
- R77: footprint Resistor_SMD:R_0201_0603Metric -> lib:R_0201_0603Metric
- TP7, TP8: footprint TestPoint:TestPoint_Pad_D1.0mm -> lib:TestPoint_Pad_D1.0mm
- U10: footprint 4in1ESC:QFN-28_L4.0-W4.0-P0.40-TL-EP2.4 -> lib:QFN-28_L4.0-W4.0-P0.40-TL-EP2.4; symbol ESCLibrary:AT32F421G8U7 -> lib:AT32F421G8U7
- U11: footprint 4in1ESC:QFN-24_L4.0-W4.0-P0.50-TL-EP2.8 -> lib:QFN-24_L4.0-W4.0-P0.50-TL-EP2.8; symbol components:NSG2065Q -> lib:NSG2065Q

Commit message: One board from the owner's 2026-08-22 Base and Core, BMP580 baro (#26)
The board is rebuilt from d81e559 (the hand-routed Base recovered from KiCad
local history and the hand-routed Core of 1fe3d21) plus the always-on +10V of
9aba717, instead of the agent-reworked 8fa8d7b. Both layouts sit side by side
in hardware/OpenAIO.kicad_pcb with all routing kept (2513 tracks, 1577 vias),
on the OpenAIO-Whoop 8L HDI stackup.

- Schematic: Core_Interface (J90/J91 LGA) removed; U26 BMP580 + C107/C108 on
  I2C0 at 0x47 (Betaflight BMP5xx default). Netlist otherwise identical to
  9aba717; ERC 31 errors, the 9aba717 baseline.
- Board: Base netclasses and severities; rule area "Core layout" keeps the
  Core's 0.09 line standard. DRC: 3 errors (USB1 peg), 37 unconnected (links).
- lib.pretty footprints replaced by the board instances; BMP580 imported with
  easyeda2kicad (LCSC C22391138).
- Not carried from 8fa8d7b: TXU0101 LED-strip buffer, +3V3_ESC, SWD pads,
  DFM edits; firmware ISSUES I2/I3 reopened.
- Docs: README pinout re-measured, AGENTS.md, research/ROUTING.md, Betaflight
  target USE_BARO_BMP580.

Co-authored-by: Stan <stan@openaio.local>
Co-authored-by: Claude Opus 5.5 <noreply@anthropic.com>
Parts:
- C35, C39, C83: Manufacturer Samsung Electro-Mechanics -> (none)
- C78, C79, C80, C88: Manufacturer Murata Electronics -> (none)
- C96, C97, C98: value 4.7uF 50v -> C; LCSC C98192 -> (none); MPN CL21A475KBQNNNE -> (none); Manufacturer Samsung Electro-Mechanics -> (none)
- Q19, Q20, Q21, Q22, Q23, Q24: footprint lib:DOY180N03T_TDFN3333-8 -> lib:Diodes_PowerDI3333-8; Manufacturer DOINGTER -> (none)
- R55, R56, R60, R61, R62, R63, R65, R68, R71: Manufacturer UNI-ROYAL -> (none)
- R57, R58, R59, R64, R66, R67, R69, R70, R72, R77: Manufacturer YAGEO -> (none)
- U11: Manufacturer NSIC -> (none)
Connections:
- net +3V3_ESC renamed +3V3
Other:
- title: ESC channel -> (none)

Commit message: Library: every symbol, footprint and 3D model project-local (#28)
* Owner: board cleanup, Core placed on the board

Co-Authored-By: Claude Opus 5.5 <noreply@anthropic.com>

* Library: every symbol, footprint and 3D model project-local

- 3D models: 275 board model paths and 28 lib.pretty footprints pointed at
  KiCad's stock install or at ${OPENDRONE_LIB} (which this machine's KiCad sets
  to a path that does not exist, so 9 models were missing). All now resolve to
  ${KIPRJMOD}/lib.3dshapes; the three missing ones come from the repo's
  KiCad-Library submodule. .wrl replaced by the .step sibling where one exists.
- Symbols: the 14 stock symbols (Device, power, Connector, Connector_Generic,
  MCU_Espressif) copied into lib.kicad_sym from the schematic's own cache and
  relinked as lib:. Four lib symbols refreshed from the schematic (they still
  held the 8fa8d7b copies).
- Pruned: 11 unused footprints, 7 unused symbols, unreferenced model files.
- tools/localise_models.py and tools/localise_symbols.py keep it that way.
- Checks: board diff is model lines only; netlist identical; ERC 31 errors as
  before, lib_symbol_mismatch 9 -> 0.

Co-Authored-By: Claude Opus 5.5 <noreply@anthropic.com>

---------

Co-authored-by: Stan <stan@openaio.local>
Co-authored-by: Claude Opus 5.5 <noreply@anthropic.com>
Parts:
- C96, C97, C98: symbol Device:C -> lib:C
- R77: symbol Device:R -> lib:R
- TP7, TP8: symbol Connector:TestPoint -> lib:TestPoint
Changed lines of the file:
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@@
 	)
 	(symbol
-		(lib_id "power:+BATT")
+		(lib_id "lib:+BATT")
 		(at 234.95 35.56 0)
 		(unit 1)
@@
 	)
 	(symbol
-		(lib_id "power:GND")
+		(lib_id "lib:GND")
 		(at 72.39 113.03 0)
 		(unit 1)
@@
 	)
 	(symbol
-		(lib_id "Connector:TestPoint")
+		(lib_id "lib:TestPoint")
 		(at 34.29 74.93 90)
 		(unit 1)
@@
 	)
 	(symbol
-		(lib_id "power:GND")
+		(lib_id "lib:GND")
 		(at 254 116.84 0)
 		(unit 1)
@@
 	)
 	(symbol
-		(lib_id "power:GND")
+		(lib_id "lib:GND")
 		(at 245.745 43.18 0)
 		(unit 1)
@@
 	)
 	(symbol
-		(lib_id "power:GND")
+		(lib_id "lib:GND")
 		(at 39.37 170.18 0)
 		(unit 1)
@@
 	)
 	(symbol
-		(lib_id "power:+BATT")
+		(lib_id "lib:+BATT")
 		(at 99.06 135.89 0)
 		(unit 1)
@@
 	)
 	(symbol
-		(lib_id "power:+BATT")
+		(lib_id "lib:+BATT")
 		(at 223.52 35.56 0)
 		(unit 1)
@@
 	)
 	(symbol
-		(lib_id "power:GND")
+		(lib_id "lib:GND")
 		(at 234.95 43.18 0)
 		(unit 1)
@@
 	)
 	(symbol
-		(lib_id "power:GND")
+		(lib_id "lib:GND")
 		(at 99.06 170.18 0)
 		(unit 1)
@@
 	)
 	(symbol
-		(lib_id "power:GND")
+		(lib_id "lib:GND")
 		(at 205.74 116.84 0)
 		(unit 1)
@@
 	)
 	(symbol
-		(lib_id "Device:C")
+		(lib_id "lib:C")
 		(at 245.745 39.37 0)
 		(unit 1)
@@
 	)
 	(symbol
-		(lib_id "power:GND")
+		(lib_id "lib:GND")
 		(at 62.23 40.64 0)
 		(unit 1)
@@
 	)
 	(symbol
-		(lib_id "power:GND")
+		(lib_id "lib:GND")
 		(at 123.19 48.26 270)
 		(unit 1)
@@
 	)
 	(symbol
-		(lib_id "power:+3V3")
+		(lib_id "lib:+3V3")
 		(at 29.21 54.61 0)
 		(unit 1)
@@
 	)
 	(symbol
-		(lib_id "power:GND")
+		(lib_id "lib:GND")
 		(at 223.52 43.18 0)
 		(unit 1)
@@
 	)
 	(symbol
-		(lib_id "Device:C")
+		(lib_id "lib:C")
 		(at 234.95 39.37 0)
 		(unit 1)
@@
 	)
 	(symbol
-		(lib_id "power:+12V")
+		(lib_id "lib:+12V")
 		(at 187.96 22.86 0)
 		(unit 1)
@@
 	)
 	(symbol
-		(lib_id "power:GND")
+		(lib_id "lib:GND")
 		(at 229.87 116.84 0)
 		(unit 1)
@@
 	)
 	(symbol
-		(lib_id "power:+BATT")
+		(lib_id "lib:+BATT")
 		(at 245.745 35.56 0)
 		(unit 1)
@@
 	)
 	(symbol
-		(lib_id "power:+3V3")
+		(lib_id "lib:+3V3")
 		(at 92.71 33.02 0)
 		(unit 1)
@@
 	)
 	(symbol
-		(lib_id "power:GND")
+		(lib_id "lib:GND")
 		(at 187.96 30.48 0)
 		(unit 1)
@@
 	)
 	(symbol
-		(lib_id "power:+12V")
+		(lib_id "lib:+12V")
 		(at 143.51 45.72 0)
 		(unit 1)
@@
 	)
 	(symbol
-		(lib_id "Device:R")
+		(lib_id "lib:R")
 		(at 71.12 33.02 90)
 		(unit 1)
@@
 	)
 	(symbol
-		(lib_id "Device:C")
+		(lib_id "lib:C")
 		(at 223.52 39.37 0)
 		(unit 1)
@@
 	)
 	(symbol
-		(lib_id "power:GND")
+		(lib_id "lib:GND")
 		(at 123.19 50.8 270)
 		(unit 1)
@@
 	)
 	(symbol
-		(lib_id "Connector:TestPoint")
+		(lib_id "lib:TestPoint")
 		(at 34.29 76.2 90)
 		(unit 1)
@@
 	)
 	(symbol
-		(lib_id "power:GND")
+		(lib_id "lib:GND")
 		(at 160.02 170.18 0)
 		(unit 1)
@@
 	)
 	(symbol
-		(lib_id "power:GND")
+		(lib_id "lib:GND")
 		(at 44.45 60.96 270)
 		(unit 1)
@@
 	)
 	(symbol
-		(lib_id "power:GND")
+		(lib_id "lib:GND")
 		(at 83.82 40.64 0)
 		(unit 1)
@@
 	)
 	(symbol
-		(lib_id "power:GND")
+		(lib_id "lib:GND")
 		(at 45.72 71.12 0)
 		(unit 1)

Commit message: Owner: rerouting in progress; KiCad re-save of the sheets (netlist unchanged)
Co-Authored-By: Claude Opus 5.5 <noreply@anthropic.com>
Parts:
- renumbered C80 to C37, C78 to C38, C79 to C39, C83 to C40, C35 to C41, C39 to C42, C88 to C43, C96 to C90, C97 to C91, C98 to C92, Q19 to Q3, Q20 to Q4, Q21 to Q5, Q22 to Q6, Q23 to Q7, Q24 to Q8, R55 to R35, R56 to R36, R57 to R37, R58 to R38, R59 to R39, R77 to R40, R60 to R41, R61 to R42, R62 to R43, R63 to R44, R64 to R45, R65 to R46, R66 to R47, R67 to R48, R68 to R49, R69 to R50, R70 to R51, R71 to R52, R72 to R53, TP7 to TP1, TP8 to TP2, U10 to U13, U11 to U14

Commit message: One 3.3 V rail: U7 becomes TLV76733DRVR (1 A), U23 removed
- U7 LP5912-3.3DRVR (500 mA) -> TLV76733DRVR (1 A, LCSC C2848334, as on
  OpenESC-20x20), same WSON-6 2x2 land; SNS (pin 2) tied to OUT in the
  schematic and by a 0.25 mm jumper on B.Cu.
- U23 TLV75533 removed; the 17 +3V3 power symbols are +3.3V, and the board's
  +3V3 copper (24 tracks, 6 vias, 3 pours) moved onto +3.3V.
- Netlist: only U7 (value, MPN, LCSC, pin 2), U23 gone, +3V3 merged into +3.3V.
  ERC 31 errors as before. DRC: no new unconnected beyond the link the old
  +3V3 side now needs to U7.
- Docs: ROUTING.md rails and reroute step; firmware notes on the single rail
  (ISSUES I15 resolved).

Co-Authored-By: Claude Opus 5.5 <noreply@anthropic.com>
Parts:
- renumbered C41 to C35, C42 to C39, C38 to C78, C39 to C79, C37 to C80, C40 to C83, C43 to C88, C90 to C96, C91 to C97, C92 to C98, Q3 to Q19, Q4 to Q20, Q5 to Q21, Q6 to Q22, Q7 to Q23, Q8 to Q24, R35 to R55, R36 to R56, R37 to R57, R38 to R58, R39 to R59, R41 to R60, R42 to R61, R43 to R62, R44 to R63, R45 to R64, R46 to R65, R47 to R66, R48 to R67, R49 to R68, R50 to R69, R51 to R70, R52 to R71, R53 to R72, R40 to R77, TP1 to TP7, TP2 to TP8, U13 to U10, U14 to U11
Connections:
- net +3V3 renamed +3.3V
Changed lines of the file:
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@@
 		(dnp no)
 		(fields_autoplaced yes)
-		(property "Reference" "R50"
+		(property "Reference" "R69"
 			(at 234.95 93.1978 0)
 			(show_name no)
@@
 		(dnp no)
 		(fields_autoplaced yes)
-		(property "Reference" "#PWR0248"
+		(property "Reference" "#PWR0260"
 			(at 234.95 39.37 0)
 			(hide yes)
@@
 		(dnp no)
 		(fields_autoplaced yes)
-		(property "Reference" "#PWR0138"
+		(property "Reference" "#PWR093"
 			(at 72.39 119.38 0)
 			(hide yes)
@@
 		(in_pos_files yes)
 		(dnp no)
-		(property "Reference" "TP1"
+		(property "Reference" "TP7"
 			(at 25.146 74.422 90)
 			(show_name no)
@@
 		(dnp no)
 		(fields_autoplaced yes)
-		(property "Reference" "#PWR0151"
+		(property "Reference" "#PWR0105"
 			(at 254 123.19 0)
 			(hide yes)
@@
 		(dnp no)
 		(fields_autoplaced yes)
-		(property "Reference" "R49"
+		(property "Reference" "R68"
 			(at 234.95 111.7599 90)
 			(show_name no)
@@
 		(dnp no)
 		(fields_autoplaced yes)
-		(property "Reference" "#PWR0251"
+		(property "Reference" "#PWR0263"
 			(at 245.745 49.53 0)
 			(hide yes)
@@
 		(in_pos_files yes)
 		(dnp no)
-		(property "Reference" "C37"
+		(property "Reference" "C80"
 			(at 41.656 69.596 0)
 			(show_name no)
@@
 		(dnp no)
 		(fields_autoplaced yes)
-		(property "Reference" "#PWR0134"
+		(property "Reference" "#PWR090"
 			(at 39.37 176.53 0)
 			(hide yes)
@@
 		(dnp no)
 		(fields_autoplaced yes)
-		(property "Reference" "#PWR0141"
+		(property "Reference" "#PWR095"
 			(at 99.06 139.7 0)
 			(hide yes)
@@
 		(dnp no)
 		(fields_autoplaced yes)
-		(property "Reference" "#PWR0246"
+		(property "Reference" "#PWR0258"
 			(at 223.52 39.37 0)
 			(hide yes)
@@
 		(dnp no)
 		(fields_autoplaced yes)
-		(property "Reference" "#PWR0249"
+		(property "Reference" "#PWR0261"
 			(at 234.95 49.53 0)
 			(hide yes)
@@
 		(in_pos_files yes)
 		(dnp no)
-		(property "Reference" "R35"
+		(property "Reference" "R55"
 			(at 29.21 142.494 90)
 			(show_name no)
@@
 		(in_pos_files yes)
 		(dnp no)
-		(property "Reference" "C41"
+		(property "Reference" "C35"
 			(at 159.004 61.976 0)
 			(show_name no)
@@
 		(dnp no)
 		(fields_autoplaced yes)
-		(property "Reference" "#PWR0142"
+		(property "Reference" "#PWR096"
 			(at 99.06 176.53 0)
 			(hide yes)
@@
 		(dnp no)
 		(fields_autoplaced yes)
-		(property "Reference" "U14"
+		(property "Reference" "U11"
 			(at 133.35 40.64 0)
 			(show_name no)
@@
 		(dnp no)
 		(fields_autoplaced yes)
-		(property "Reference" "#PWR0149"
+		(property "Reference" "#PWR0103"
 			(at 205.74 123.19 0)
 			(hide yes)
@@
 		(dnp no)
 		(fields_autoplaced yes)
-		(property "Reference" "R45"
+		(property "Reference" "R64"
 			(at 210.82 90.1699 90)
 			(show_name no)
@@
 		(dnp no)
 		(fields_autoplaced yes)
-		(property "Reference" "C92"
+		(property "Reference" "C98"
 			(at 248.92 38.0999 0)
 			(show_name no)
@@
 		(in_pos_files yes)
 		(dnp no)
-		(property "Reference" "#PWR0137"
+		(property "Reference" "#PWR086"
 			(at 62.23 46.99 0)
 			(hide yes)
@@
 		(dnp no)
 		(fields_autoplaced yes)
-		(property "Reference" "R47"
+		(property "Reference" "R66"
 			(at 210.82 92.71 0)
 			(show_name no)
@@
 		(in_pos_files yes)
 		(dnp no)
-		(property "Reference" "#PWR0143"
+		(property "Reference" "#PWR097"
 			(at 116.84 48.26 0)
 			(hide yes)
@@
 		(in_pos_files yes)
 		(dnp no)
-		(property "Reference" "C39"
+		(property "Reference" "C79"
 			(at 80.264 35.814 90)
 			(show_name no)
@@
 		(dnp no)
 		(fields_autoplaced yes)
-		(property "Reference" "R38"
+		(property "Reference" "R58"
 			(at 49.53 54.61 0)
 			(show_name no)
@@
 		(dnp no)
 		(fields_autoplaced yes)
-		(property "Reference" "R53"
+		(property "Reference" "R72"
 			(at 259.08 92.71 0)
 			(show_name no)
@@
 		(in_pos_files yes)
 		(dnp no)
-		(property "Reference" "C38"
+		(property "Reference" "C78"
 			(at 58.166 39.116 0)
 			(show_name no)
@@
 		(dnp no)
 		(fields_autoplaced yes)
-		(property "Reference" "R46"
+		(property "Reference" "R65"
 			(at 210.82 111.7599 90)
 			(show_name no)
@@
 		(dnp no)
 		(fields_autoplaced yes)
-		(property "Reference" "R51"
+		(property "Reference" "R70"
 			(at 256.54 90.1699 90)
 			(show_name no)
@@
 		(in_pos_files yes)
 		(dnp no)
-		(property "Reference" "C40"
+		(property "Reference" "C83"
 			(at 148.844 59.436 0)
 			(show_name no)
@@
 		(dnp no)
 		(fields_autoplaced yes)
-		(property "Reference" "R48"
+		(property "Reference" "R67"
 			(at 232.41 90.1699 90)
 			(show_name no)
@@
 	)
 	(symbol
-		(lib_id "lib:+3V3")
+		(lib_id "lib:+3.3V")
 		(at 29.21 54.61 0)
 		(unit 1)
@@
 		(dnp no)
 		(fields_autoplaced yes)
-		(property "Reference" "#PWR0133"
+		(property "Reference" "#PWR087"
 			(at 29.21 58.42 0)
 			(hide yes)
@@
 			)
 		)
-		(property "Value" "+3V3"
+		(property "Value" "+3.3V"
 			(at 29.21 49.53 0)
 			(show_name no)
@@
 		(in_pos_files yes)
 		(dnp no)
-		(property "Reference" "R42"
+		(property "Reference" "R61"
 			(at 88.9 157.734 90)
 			(show_name no)
@@
 		(in_pos_files yes)
 		(dnp no)
-		(property "Reference" "C43"
+		(property "Reference" "C88"
 			(at 183.896 28.956 0)
 			(show_name no)
@@
 		(in_pos_files yes)
 		(dnp no)
-		(property "Reference" "U13"
+		(property "Reference" "U10"
 			(at 71.882 73.152 0)
 			(show_name no)
@@
 		(in_pos_files yes)
 		(dnp no)
-		(property "Reference" "R44"
+		(property "Reference" "R63"
 			(at 149.86 156.464 90)
 			(show_name no)
@@
 		(dnp no)
 		(fields_autoplaced yes)
-		(property "Reference" "#PWR0247"
+		(property "Reference" "#PWR0259"
 			(at 223.52 49.53 0)
 			(hide yes)
@@
 		(dnp no)
 		(fields_autoplaced yes)
-		(property "Reference" "Q5"
+		(property "Reference" "Q21"
 			(at 102.87 144.7799 0)
 			(show_name no)
@@
 		(dnp no)
 		(fields_autoplaced yes)
-		(property "Reference" "C91"
+		(property "Reference" "C97"
 			(at 238.125 38.0999 0)
 			(show_name no)
@@
 		(in_pos_files yes)
 		(dnp no)
-		(property "Reference" "R43"
+		(property "Reference" "R62"
 			(at 149.86 141.224 90)
 			(show_name no)
@@
 		(in_pos_files yes)
 		(dnp no)
-		(property "Reference" "R41"
+		(property "Reference" "R60"
 			(at 88.9 142.494 90)
 			(show_name no)
@@
 		(dnp no)
 		(fields_autoplaced yes)
-		(property "Reference" "#PWR0147"
+		(property "Reference" "#PWR059"
 			(at 187.96 26.67 0)
 			(hide yes)
@@
 		(dnp no)
 		(fields_autoplaced yes)
-		(property "Reference" "Q4"
+		(property "Reference" "Q20"
 			(at 43.18 160.0199 0)
 			(show_name no)
@@
 		(dnp no)
 		(fields_autoplaced yes)
-		(property "Reference" "R52"
+		(property "Reference" "R71"
 			(at 259.08 111.7599 90)
 			(show_name no)
@@
 		(dnp no)
 		(fields_autoplaced yes)
-		(property "Reference" "Q7"
+		(property "Reference" "Q23"
 			(at 163.83 143.5099 0)
 			(show_name no)
@@
 		(dnp no)
 		(fields_autoplaced yes)
-		(property "Reference" "#PWR0150"
+		(property "Reference" "#PWR0104"
 			(at 229.87 123.19 0)
 			(hide yes)
@@
 		(dnp no)
 		(fields_autoplaced yes)
-		(property "Reference" "#PWR0250"
+		(property "Reference" "#PWR0262"
 			(at 245.745 39.37 0)
 			(hide yes)
@@
 		(in_pos_files yes)
 		(dnp no)
-		(property "Reference" "R36"
+		(property "Reference" "R56"
 			(at 29.21 157.734 90)
 			(show_name no)
@@
 	)
 	(symbol
-		(lib_id "lib:+3V3")
+		(lib_id "lib:+3.3V")
 		(at 92.71 33.02 0)
 		(unit 1)
@@
 		(dnp no)
 		(fields_autoplaced yes)
-		(property "Reference" "#PWR0140"
+		(property "Reference" "#PWR0114"
 			(at 92.71 36.83 0)
 			(hide yes)
@@
 			)
 		)
-		(property "Value" "+3V3"
+		(property "Value" "+3.3V"
 			(at 92.71 27.94 0)
 			(show_name no)
@@
 		(in_pos_files yes)
 		(dnp no)
-		(property "Reference" "#PWR0148"
+		(property "Reference" "#PWR0102"
 			(at 187.96 36.83 0)
 			(hide yes)
@@
 		(dnp no)
 		(fields_autoplaced yes)
-		(property "Reference" "#PWR0145"
+		(property "Reference" "#PWR0101"
 			(at 143.51 49.53 0)
 			(hide yes)
@@
 		(in_pos_files yes)
 		(dnp no)
-		(property "Reference" "C42"
+		(property "Reference" "C39"
 			(at 169.164 64.516 0)
 			(show_name no)
@@
 		(dnp no)
 		(fields_autoplaced yes)
-		(property "Reference" "R40"
+		(property "Reference" "R77"
 			(at 71.12 26.67 90)
 			(show_name no)
@@
 		(dnp no)
 		(fields_autoplaced yes)
-		(property "Reference" "Q3"
+		(property "Reference" "Q19"
 			(at 43.18 144.7799 0)
 			(show_name no)
@@
 		(dnp no)
 		(fields_autoplaced yes)
-		(property "Reference" "C90"
+		(property "Reference" "C96"
 			(at 226.695 38.0999 0)
 			(show_name no)
@@
 		(dnp no)
 		(fields_autoplaced yes)
-		(property "Reference" "R39"
+		(property "Reference" "R59"
 			(at 49.7944 85.09 90)
 			(hide yes)
@@
 		(in_pos_files yes)
 		(dnp no)
-		(property "Reference" "#PWR0144"
+		(property "Reference" "#PWR098"
 			(at 116.84 50.8 0)
 			(hide yes)
@@
 		(in_pos_files yes)
 		(dnp no)
-		(property "Reference" "TP2"
+		(property "Reference" "TP8"
 			(at 25.146 76.708 90)
 			(show_name no)
@@
 		(dnp no)
 		(fields_autoplaced yes)
-		(property "Reference" "#PWR0146"
+		(property "Reference" "#PWR0100"
 			(at 160.02 176.53 0)
 			(hide yes)
@@
 		(dnp no)
 		(fields_autoplaced yes)
-		(property "Reference" "R37"
+		(property "Reference" "R57"
 			(at 34.29 57.15 0)
 			(show_name no)
@@
 		(in_pos_files yes)
 		(dnp no)
-		(property "Reference" "#PWR0135"
+		(property "Reference" "#PWR091"
 			(at 38.1 60.96 0)
 			(hide yes)
@@
 		(in_pos_files yes)
 		(dnp no)
-		(property "Reference" "#PWR0139"
+		(property "Reference" "#PWR089"
 			(at 83.82 46.99 0)
 			(hide yes)
@@
 		(in_pos_files yes)
 		(dnp no)
-		(property "Reference" "#PWR0136"
+		(property "Reference" "#PWR092"
 			(at 45.72 77.47 0)
 			(hide yes)
@@
 		(dnp no)
 		(fields_autoplaced yes)
-		(property "Reference" "Q6"
+		(property "Reference" "Q22"
 			(at 102.87 160.0199 0)
 			(show_name no)
@@
 		(dnp no)
 		(fields_autoplaced yes)
-		(property "Reference" "Q8"
+		(property "Reference" "Q24"
 			(at 163.83 158.7499 0)
 			(show_name no)
