File: hardware/esc_channel.kicad_sch (KiCad schematic)
At the start: 39 parts, among them Q19 DOY180N03T, Q20 DOY180N03T, Q21 DOY180N03T, Q22 DOY180N03T, Q23 DOY180N03T, Q24 DOY180N03T, U10 AT32F421G8U7, U11 NSG2065Q

Commit message: Owner: routing in progress
Co-Authored-By: Claude Opus 5.5 <noreply@anthropic.com>
Parts:
- renumbered C80 to C37, C78 to C38, C79 to C39, C83 to C40, C35 to C41, C39 to C42, C88 to C43, C96 to C90, C97 to C91, C98 to C92, Q19 to Q3, Q20 to Q4, Q21 to Q5, Q22 to Q6, Q23 to Q7, Q24 to Q8, R55 to R35, R56 to R36, R57 to R37, R58 to R38, R59 to R39, R77 to R40, R60 to R41, R61 to R42, R62 to R43, R63 to R44, R64 to R45, R65 to R46, R66 to R47, R67 to R48, R68 to R49, R69 to R50, R70 to R51, R71 to R52, R72 to R53, TP7 to TP1, TP8 to TP2, U10 to U13, U11 to U14
Changed lines of the file:
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@@
 		(dnp no)
 		(fields_autoplaced yes)
-		(property "Reference" "R69"
+		(property "Reference" "R50"
 			(at 234.95 93.1978 0)
 			(show_name no)
@@
 		(dnp no)
 		(fields_autoplaced yes)
-		(property "Reference" "#PWR0260"
+		(property "Reference" "#PWR0248"
 			(at 234.95 39.37 0)
 			(hide yes)
@@
 		(dnp no)
 		(fields_autoplaced yes)
-		(property "Reference" "#PWR093"
+		(property "Reference" "#PWR0138"
 			(at 72.39 119.38 0)
 			(hide yes)
@@
 		(in_pos_files yes)
 		(dnp no)
-		(property "Reference" "TP7"
+		(property "Reference" "TP1"
 			(at 25.146 74.422 90)
 			(show_name no)
@@
 		(dnp no)
 		(fields_autoplaced yes)
-		(property "Reference" "#PWR0105"
+		(property "Reference" "#PWR0151"
 			(at 254 123.19 0)
 			(hide yes)
@@
 		(dnp no)
 		(fields_autoplaced yes)
-		(property "Reference" "R68"
+		(property "Reference" "R49"
 			(at 234.95 111.7599 90)
 			(show_name no)
@@
 		(dnp no)
 		(fields_autoplaced yes)
-		(property "Reference" "#PWR0263"
+		(property "Reference" "#PWR0251"
 			(at 245.745 49.53 0)
 			(hide yes)
@@
 		(in_pos_files yes)
 		(dnp no)
-		(property "Reference" "C80"
+		(property "Reference" "C37"
 			(at 41.656 69.596 0)
 			(show_name no)
@@
 		(dnp no)
 		(fields_autoplaced yes)
-		(property "Reference" "#PWR090"
+		(property "Reference" "#PWR0134"
 			(at 39.37 176.53 0)
 			(hide yes)
@@
 		(dnp no)
 		(fields_autoplaced yes)
-		(property "Reference" "#PWR095"
+		(property "Reference" "#PWR0141"
 			(at 99.06 139.7 0)
 			(hide yes)
@@
 		(dnp no)
 		(fields_autoplaced yes)
-		(property "Reference" "#PWR0258"
+		(property "Reference" "#PWR0246"
 			(at 223.52 39.37 0)
 			(hide yes)
@@
 		(dnp no)
 		(fields_autoplaced yes)
-		(property "Reference" "#PWR0261"
+		(property "Reference" "#PWR0249"
 			(at 234.95 49.53 0)
 			(hide yes)
@@
 		(in_pos_files yes)
 		(dnp no)
-		(property "Reference" "R55"
+		(property "Reference" "R35"
 			(at 29.21 142.494 90)
 			(show_name no)
@@
 		(in_pos_files yes)
 		(dnp no)
-		(property "Reference" "C35"
+		(property "Reference" "C41"
 			(at 159.004 61.976 0)
 			(show_name no)
@@
 		(dnp no)
 		(fields_autoplaced yes)
-		(property "Reference" "#PWR096"
+		(property "Reference" "#PWR0142"
 			(at 99.06 176.53 0)
 			(hide yes)
@@
 		(dnp no)
 		(fields_autoplaced yes)
-		(property "Reference" "U11"
+		(property "Reference" "U14"
 			(at 133.35 40.64 0)
 			(show_name no)
@@
 		(dnp no)
 		(fields_autoplaced yes)
-		(property "Reference" "#PWR0103"
+		(property "Reference" "#PWR0149"
 			(at 205.74 123.19 0)
 			(hide yes)
@@
 		(dnp no)
 		(fields_autoplaced yes)
-		(property "Reference" "R64"
+		(property "Reference" "R45"
 			(at 210.82 90.1699 90)
 			(show_name no)
@@
 		(dnp no)
 		(fields_autoplaced yes)
-		(property "Reference" "C98"
+		(property "Reference" "C92"
 			(at 248.92 38.0999 0)
 			(show_name no)
@@
 		(in_pos_files yes)
 		(dnp no)
-		(property "Reference" "#PWR086"
+		(property "Reference" "#PWR0137"
 			(at 62.23 46.99 0)
 			(hide yes)
@@
 		(dnp no)
 		(fields_autoplaced yes)
-		(property "Reference" "R66"
+		(property "Reference" "R47"
 			(at 210.82 92.71 0)
 			(show_name no)
@@
 		(in_pos_files yes)
 		(dnp no)
-		(property "Reference" "#PWR097"
+		(property "Reference" "#PWR0143"
 			(at 116.84 48.26 0)
 			(hide yes)
@@
 		(in_pos_files yes)
 		(dnp no)
-		(property "Reference" "C79"
+		(property "Reference" "C39"
 			(at 80.264 35.814 90)
 			(show_name no)
@@
 		(dnp no)
 		(fields_autoplaced yes)
-		(property "Reference" "R58"
+		(property "Reference" "R38"
 			(at 49.53 54.61 0)
 			(show_name no)
@@
 		(dnp no)
 		(fields_autoplaced yes)
-		(property "Reference" "R72"
+		(property "Reference" "R53"
 			(at 259.08 92.71 0)
 			(show_name no)
@@
 		(in_pos_files yes)
 		(dnp no)
-		(property "Reference" "C78"
+		(property "Reference" "C38"
 			(at 58.166 39.116 0)
 			(show_name no)
@@
 		(dnp no)
 		(fields_autoplaced yes)
-		(property "Reference" "R65"
+		(property "Reference" "R46"
 			(at 210.82 111.7599 90)
 			(show_name no)
@@
 		(dnp no)
 		(fields_autoplaced yes)
-		(property "Reference" "R70"
+		(property "Reference" "R51"
 			(at 256.54 90.1699 90)
 			(show_name no)
@@
 		(in_pos_files yes)
 		(dnp no)
-		(property "Reference" "C83"
+		(property "Reference" "C40"
 			(at 148.844 59.436 0)
 			(show_name no)
@@
 		(dnp no)
 		(fields_autoplaced yes)
-		(property "Reference" "R67"
+		(property "Reference" "R48"
 			(at 232.41 90.1699 90)
 			(show_name no)
@@
 		(dnp no)
 		(fields_autoplaced yes)
-		(property "Reference" "#PWR087"
+		(property "Reference" "#PWR0133"
 			(at 29.21 58.42 0)
 			(hide yes)
@@
 		(in_pos_files yes)
 		(dnp no)
-		(property "Reference" "R61"
+		(property "Reference" "R42"
 			(at 88.9 157.734 90)
 			(show_name no)
@@
 		(in_pos_files yes)
 		(dnp no)
-		(property "Reference" "C88"
+		(property "Reference" "C43"
 			(at 183.896 28.956 0)
 			(show_name no)
@@
 		(in_pos_files yes)
 		(dnp no)
-		(property "Reference" "U10"
+		(property "Reference" "U13"
 			(at 71.882 73.152 0)
 			(show_name no)
@@
 		(in_pos_files yes)
 		(dnp no)
-		(property "Reference" "R63"
+		(property "Reference" "R44"
 			(at 149.86 156.464 90)
 			(show_name no)
@@
 		(dnp no)
 		(fields_autoplaced yes)
-		(property "Reference" "#PWR0259"
+		(property "Reference" "#PWR0247"
 			(at 223.52 49.53 0)
 			(hide yes)
@@
 		(dnp no)
 		(fields_autoplaced yes)
-		(property "Reference" "Q21"
+		(property "Reference" "Q5"
 			(at 102.87 144.7799 0)
 			(show_name no)
@@
 		(dnp no)
 		(fields_autoplaced yes)
-		(property "Reference" "C97"
+		(property "Reference" "C91"
 			(at 238.125 38.0999 0)
 			(show_name no)
@@
 		(in_pos_files yes)
 		(dnp no)
-		(property "Reference" "R62"
+		(property "Reference" "R43"
 			(at 149.86 141.224 90)
 			(show_name no)
@@
 		(in_pos_files yes)
 		(dnp no)
-		(property "Reference" "R60"
+		(property "Reference" "R41"
 			(at 88.9 142.494 90)
 			(show_name no)
@@
 		(dnp no)
 		(fields_autoplaced yes)
-		(property "Reference" "#PWR059"
+		(property "Reference" "#PWR0147"
 			(at 187.96 26.67 0)
 			(hide yes)
@@
 		(dnp no)
 		(fields_autoplaced yes)
-		(property "Reference" "Q20"
+		(property "Reference" "Q4"
 			(at 43.18 160.0199 0)
 			(show_name no)
@@
 		(dnp no)
 		(fields_autoplaced yes)
-		(property "Reference" "R71"
+		(property "Reference" "R52"
 			(at 259.08 111.7599 90)
 			(show_name no)
@@
 		(dnp no)
 		(fields_autoplaced yes)
-		(property "Reference" "Q23"
+		(property "Reference" "Q7"
 			(at 163.83 143.5099 0)
 			(show_name no)
@@
 		(dnp no)
 		(fields_autoplaced yes)
-		(property "Reference" "#PWR0104"
+		(property "Reference" "#PWR0150"
 			(at 229.87 123.19 0)
 			(hide yes)
@@
 		(dnp no)
 		(fields_autoplaced yes)
-		(property "Reference" "#PWR0262"
+		(property "Reference" "#PWR0250"
 			(at 245.745 39.37 0)
 			(hide yes)
@@
 		(in_pos_files yes)
 		(dnp no)
-		(property "Reference" "R56"
+		(property "Reference" "R36"
 			(at 29.21 157.734 90)
 			(show_name no)
@@
 		(dnp no)
 		(fields_autoplaced yes)
-		(property "Reference" "#PWR0114"
+		(property "Reference" "#PWR0140"
 			(at 92.71 36.83 0)
 			(hide yes)
@@
 		(in_pos_files yes)
 		(dnp no)
-		(property "Reference" "#PWR0102"
+		(property "Reference" "#PWR0148"
 			(at 187.96 36.83 0)
 			(hide yes)
@@
 		(dnp no)
 		(fields_autoplaced yes)
-		(property "Reference" "#PWR0101"
+		(property "Reference" "#PWR0145"
 			(at 143.51 49.53 0)
 			(hide yes)
@@
 		(in_pos_files yes)
 		(dnp no)
-		(property "Reference" "C39"
+		(property "Reference" "C42"
 			(at 169.164 64.516 0)
 			(show_name no)
@@
 		(dnp no)
 		(fields_autoplaced yes)
-		(property "Reference" "R77"
+		(property "Reference" "R40"
 			(at 71.12 26.67 90)
 			(show_name no)
@@
 		(dnp no)
 		(fields_autoplaced yes)
-		(property "Reference" "Q19"
+		(property "Reference" "Q3"
 			(at 43.18 144.7799 0)
 			(show_name no)
@@
 		(dnp no)
 		(fields_autoplaced yes)
-		(property "Reference" "C96"
+		(property "Reference" "C90"
 			(at 226.695 38.0999 0)
 			(show_name no)
@@
 		(dnp no)
 		(fields_autoplaced yes)
-		(property "Reference" "R59"
+		(property "Reference" "R39"
 			(at 49.7944 85.09 90)
 			(hide yes)
@@
 		(in_pos_files yes)
 		(dnp no)
-		(property "Reference" "#PWR098"
+		(property "Reference" "#PWR0144"
 			(at 116.84 50.8 0)
 			(hide yes)
@@
 		(in_pos_files yes)
 		(dnp no)
-		(property "Reference" "TP8"
+		(property "Reference" "TP2"
 			(at 25.146 76.708 90)
 			(show_name no)
@@
 		(dnp no)
 		(fields_autoplaced yes)
-		(property "Reference" "#PWR0100"
+		(property "Reference" "#PWR0146"
 			(at 160.02 176.53 0)
 			(hide yes)
@@
 		(dnp no)
 		(fields_autoplaced yes)
-		(property "Reference" "R57"
+		(property "Reference" "R37"
 			(at 34.29 57.15 0)
 			(show_name no)
@@
 		(in_pos_files yes)
 		(dnp no)
-		(property "Reference" "#PWR091"
+		(property "Reference" "#PWR0135"
 			(at 38.1 60.96 0)
 			(hide yes)
@@
 		(in_pos_files yes)
 		(dnp no)
-		(property "Reference" "#PWR089"
+		(property "Reference" "#PWR0139"
 			(at 83.82 46.99 0)
 			(hide yes)
@@
 		(in_pos_files yes)
 		(dnp no)
-		(property "Reference" "#PWR092"
+		(property "Reference" "#PWR0136"
 			(at 45.72 77.47 0)
 			(hide yes)
@@
 		(dnp no)
 		(fields_autoplaced yes)
-		(property "Reference" "Q22"
+		(property "Reference" "Q6"
 			(at 102.87 160.0199 0)
 			(show_name no)
@@
 		(dnp no)
 		(fields_autoplaced yes)
-		(property "Reference" "Q24"
+		(property "Reference" "Q8"
 			(at 163.83 158.7499 0)
 			(show_name no)
