File: hardware/fc_imu.kicad_sch (KiCad schematic)
At the start: 4 parts, among them U9 BMI270

Commit message: Net classes: VBAT, Phase, Power, Gate, USB, RF, Analog with colours and patterns
Replaces the stale 50Ohm /ELRS/* patterns inherited from the template.
Widths and clearances start from the line standard (0.09/0.09, via 0.35/0.20)
and the ESC boards' practice; USB and RF geometry still to be checked against
the chosen JLCPCB 6-layer stackup.
Parts:
- renumbered C35 to C29, C36 to C30, R49 to R25, U9 to U8
Changed lines of the file:
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@@
 		(in_pos_files yes)
 		(dnp no)
-		(property "Reference" "R49"
+		(property "Reference" "R25"
 			(at 106.172 75.946 90)
 			(show_name no)
@@
 			(project "OpenAIO"
 				(path "/fb88b6f9-ee39-4640-a9d4-04a17ceeac64/067dfe4f-0feb-4fee-b449-2d51932eecf1"
-					(reference "R49")
+					(reference "R25")
 					(unit 1)
 				)
@@
 		(dnp no)
 		(fields_autoplaced yes)
-		(property "Reference" "#PWR0130"
+		(property "Reference" "#PWR080"
 			(at 83.82 46.99 0)
 			(hide yes)
@@
 			(project "OpenAIO"
 				(path "/fb88b6f9-ee39-4640-a9d4-04a17ceeac64/067dfe4f-0feb-4fee-b449-2d51932eecf1"
-					(reference "#PWR0130")
+					(reference "#PWR080")
 					(unit 1)
 				)
@@
 		(dnp no)
 		(fields_autoplaced yes)
-		(property "Reference" "#PWR0156"
+		(property "Reference" "#PWR082"
 			(at 107.95 78.74 0)
 			(hide yes)
@@
 			(project "OpenAIO"
 				(path "/fb88b6f9-ee39-4640-a9d4-04a17ceeac64/067dfe4f-0feb-4fee-b449-2d51932eecf1"
-					(reference "#PWR0156")
+					(reference "#PWR082")
 					(unit 1)
 				)
@@
 		(dnp no)
 		(fields_autoplaced yes)
-		(property "Reference" "#PWR0125"
+		(property "Reference" "#PWR076"
 			(at 45.72 99.06 0)
 			(hide yes)
@@
 			(project "OpenAIO"
 				(path "/fb88b6f9-ee39-4640-a9d4-04a17ceeac64/067dfe4f-0feb-4fee-b449-2d51932eecf1"
-					(reference "#PWR0125")
+					(reference "#PWR076")
 					(unit 1)
 				)
@@
 		(dnp no)
 		(fields_autoplaced yes)
-		(property "Reference" "#PWR0131"
+		(property "Reference" "#PWR081"
 			(at 83.82 57.15 0)
 			(hide yes)
@@
 			(project "OpenAIO"
 				(path "/fb88b6f9-ee39-4640-a9d4-04a17ceeac64/067dfe4f-0feb-4fee-b449-2d51932eecf1"
-					(reference "#PWR0131")
+					(reference "#PWR081")
 					(unit 1)
 				)
@@
 		(in_pos_files yes)
 		(dnp no)
-		(property "Reference" "C35"
+		(property "Reference" "C29"
 			(at 62.23 44.45 0)
 			(show_name no)
@@
 			(project "OpenAIO"
 				(path "/fb88b6f9-ee39-4640-a9d4-04a17ceeac64/067dfe4f-0feb-4fee-b449-2d51932eecf1"
-					(reference "C35")
+					(reference "C29")
 					(unit 1)
 				)
@@
 		(dnp no)
 		(fields_autoplaced yes)
-		(property "Reference" "#PWR0127"
+		(property "Reference" "#PWR077"
 			(at 62.23 46.99 0)
 			(hide yes)
@@
 			(project "OpenAIO"
 				(path "/fb88b6f9-ee39-4640-a9d4-04a17ceeac64/067dfe4f-0feb-4fee-b449-2d51932eecf1"
-					(reference "#PWR0127")
+					(reference "#PWR077")
 					(unit 1)
 				)
@@
 		(in_pos_files yes)
 		(dnp no)
-		(property "Reference" "U9"
+		(property "Reference" "U8"
 			(at 60.96 68.326 0)
 			(show_name no)
@@
 			(project "OpenAIO"
 				(path "/fb88b6f9-ee39-4640-a9d4-04a17ceeac64/067dfe4f-0feb-4fee-b449-2d51932eecf1"
-					(reference "U9")
+					(reference "U8")
 					(unit 1)
 				)
@@
 		(dnp no)
 		(fields_autoplaced yes)
-		(property "Reference" "#PWR0126"
+		(property "Reference" "#PWR078"
 			(at 62.23 57.15 0)
 			(hide yes)
@@
 			(project "OpenAIO"
 				(path "/fb88b6f9-ee39-4640-a9d4-04a17ceeac64/067dfe4f-0feb-4fee-b449-2d51932eecf1"
-					(reference "#PWR0126")
+					(reference "#PWR078")
 					(unit 1)
 				)
@@
 		(dnp no)
 		(fields_autoplaced yes)
-		(property "Reference" "#PWR0128"
+		(property "Reference" "#PWR079"
 			(at 72.39 99.06 0)
 			(hide yes)
@@
 			(project "OpenAIO"
 				(path "/fb88b6f9-ee39-4640-a9d4-04a17ceeac64/067dfe4f-0feb-4fee-b449-2d51932eecf1"
-					(reference "#PWR0128")
+					(reference "#PWR079")
 					(unit 1)
 				)
@@
 		(in_pos_files yes)
 		(dnp no)
-		(property "Reference" "C36"
+		(property "Reference" "C30"
 			(at 83.82 44.45 0)
 			(show_name no)
@@
 			(project "OpenAIO"
 				(path "/fb88b6f9-ee39-4640-a9d4-04a17ceeac64/067dfe4f-0feb-4fee-b449-2d51932eecf1"
-					(reference "C36")
-					(unit 1)
-				)
+					(reference "C30")
+					(unit 1)
+				)

Commit message: OpenAIO: master PCB with Base and Core islands routed, AIO_outline footprint+symbol in project lib
Save point before the two-board (LGA) split tooling.
Parts:
- C29, C30, R25: KiLib_Generator (none) -> SMD_2terminal_chip_molded
Changed lines of the file:
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@@
+			)
+		)
+		(property "KiLib_Generator" "SMD_2terminal_chip_molded"
+			(at 107.95 78.74 0)
+			(hide yes)
+			(show_name no)
+			(do_not_autoplace no)
+			(effects
+				(font
+					(size 1.27 1.27)
+				)
 			)
 		)
@@
 			)
 		)
+		(property "KiLib_Generator" "SMD_2terminal_chip_molded"
+			(at 62.23 46.99 0)
+			(hide yes)
+			(show_name no)
+			(do_not_autoplace no)
+			(effects
+				(font
+					(size 1.27 1.27)
+				)
+			)
+		)
 		(pin "1"
 		)
@@
 			(hide yes)
 			(show_name no)
+			(do_not_autoplace no)
+			(effects
+				(font
+					(size 1.27 1.27)
+				)
+			)
+		)
+		(property "KiLib_Generator" "SMD_2terminal_chip_molded"
+			(at 83.82 46.99 0)
+			(hide yes)
+			(show_name no)
