File: hardware/fc_imu.kicad_sch (KiCad schematic)
At the start: 4 parts, among them U8 BMI270

Commit message: Circuit: B3 bulk caps and ESP32-C3FH4, LDO caps, BMI270 aux pins, BOOTSEL 1k, unused pads
CIRCUIT_REVIEW B3, S2, S4, S5 and decision D9; LAYOUT_REVIEW 5.3 (pure
clean-up). Values and parts from hardware/KiCad-Library/PARTS-USED.md.

- B3: the 16 +BATT bulk caps had value "C" and no part. C90-C103 (0805)
  4.7uF 50V X5R CL21A475KBQNNNE (C98192, already C18/C19); C105/C106 (1206)
  4.7uF 50V X7R TCC1206X7R475K500HT (C380366, OpenESC).
- D9/B3: U22 is ESP32-C3FH4 (C2858491, in-package flash), as its NC SPI pins
  require; its in-package-flash pads 19, 21-24 deleted per instance (20 was
  already gone). L4 MPN MLZ2012M150WT000 (TDK, SX1281 reference BOM, LCSC not
  in the catalogue); D9 MPN/manufacturer/LCSC from the catalogue.
- S2, LP5912 windows (CIN > 0.5 uF effective, COUT 0.7-10 uF): U7 COUT C28
  22uF -> 1uF CL05A105KA5NQNC; U6 COUT C27 22uF -> 4.7uF CL05A475MP5NRNC;
  U7 CIN C26 100nF -> 1uF GRM033R61A105ME44D in the existing 0201 (an 0402
  does not fit beside U7 without moving parts; ~0.5 uF effective at 4.6 V,
  so it is marginal until U7 moves to the Core in R2, decision S1).
- S4: BMI270 U8 ASDx/ASCx (pins 2/3) were on GND, which the datasheet
  forbids; now +3.3V (VDDIO), valid for the LSM6DSV16X option too.
  Schematic: the GND drop replaced by a +3.3V symbol. Core: pads 2/3 and the
  via between them re-netted, 0.15 mm In3 stub to the In3 +3.3V pour.
- S5: BOOTSEL resistor R7 10k -> 1k (0201WMF1001TEE, C270365): 10k with the
  32k minimum pull-up gave 0.79 V against VIL 0.8 V.
- LAYOUT_REVIEW 5.3, pads on no net with nothing attached: U13/U15/U17/U19
  (AT32F421) 3, 8, 9, 12, 23, 24, 26-28; U14/U16/U18/U20 (NSG2065Q) NC 5, 7,
  8, 21; U7 NC 2; U21 6 (XTB, TCXO), 9, 10 (DIO2/3); Core U2 55-59 (QSPI,
  in-package flash). 60 pads in all; U8 kept for joint symmetry. AT32
  firmware must keep the dropped pins as outputs or pulled.
- Footprint values and fields synced from the schematic for the changed refs.

Deferred: RX LED D9 to +4v5 (S10). +4v5 copper is 1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
Connections:
- net +3.3V: now also U8.2 (SDx/AH1/Qvar1), U8.3 (SCx/AH2/Qvar2)
- net GND: no longer U8.2 (SDx/AH1/Qvar1), U8.3 (SCx/AH2/Qvar2)
Changed lines of the file:
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@@
-		(color 0 0 0 0)
-	)
-	(junction
-		(at 45.72 81.28)
-		(diameter 0)
 		(color 0 0 0 0)
 	)
@@
 		(pts
 			(xy 73.66 57.15) (xy 73.66 43.18)
-		)
-		(stroke
-			(width 0)
-			(type default)
-		)
-	)
-	(wire
-		(pts
-			(xy 45.72 92.71) (xy 45.72 81.28)
 		)
 		(stroke
@@
 	(symbol
 		(lib_id "power:GND")
-		(at 45.72 92.71 0)
-		(unit 1)
-		(body_style 1)
-		(exclude_from_sim no)
-		(in_bom yes)
-		(on_board yes)
-		(in_pos_files yes)
-		(dnp no)
-		(fields_autoplaced yes)
-		(property "Reference" "#PWR076"
-			(at 45.72 99.06 0)
-			(hide yes)
-			(show_name no)
-			(do_not_autoplace no)
-			(effects
-				(font
-					(size 1.27 1.27)
-				)
-			)
-		)
-		(property "Value" "GND"
-			(at 45.72 97.79 0)
-			(show_name no)
-			(do_not_autoplace no)
-			(effects
-				(font
-					(size 1.27 1.27)
-				)
-			)
-		)
-		(property "Footprint" ""
-			(at 45.72 92.71 0)
-			(hide yes)
-			(show_name no)
-			(do_not_autoplace no)
-			(effects
-				(font
-					(size 1.27 1.27)
-				)
-			)
-		)
-		(property "Datasheet" ""
-			(at 45.72 92.71 0)
-			(hide yes)
-			(show_name no)
-			(do_not_autoplace no)
-			(effects
-				(font
-					(size 1.27 1.27)
-				)
-			)
-		)
-		(property "Description" "Power symbol creates a global label with name \"GND\" , ground"
-			(at 45.72 92.71 0)
-			(hide yes)
-			(show_name no)
-			(do_not_autoplace no)
-			(effects
-				(font
-					(size 1.27 1.27)
-				)
-			)
-		)
-		(pin "1"
-		)
-		(instances
-			(project "OpenAIO-Base"
-				(path "/fb88b6f9-ee39-4640-a9d4-04a17ceeac64/067dfe4f-0feb-4fee-b449-2d51932eecf1"
-					(reference "#PWR076")
-					(unit 1)
-				)
-			)
-		)
-	)
-	(symbol
-		(lib_id "power:GND")
 		(at 83.82 50.8 0)
 		(unit 1)
@@
 					(unit 1)
 				)
+			)
+		)
+	)
+	(symbol
+		(lib_name "+3.3V_1")
+		(lib_id "power:+3.3V")
+		(at 45.72 78.74 0)
+		(unit 1)
+		(body_style 1)
+		(exclude_from_sim no)
+		(in_bom yes)
+		(on_board yes)
+		(in_pos_files yes)
+		(dnp no)
+		(fields_autoplaced yes)
+		(property "Reference" "#PWR0289"
+			(at 45.72 82.55 0)
+			(hide yes)
+			(show_name no)
+			(do_not_autoplace no)
+			(effects
+				(font
+					(size 1.27 1.27)
+				)
+			)
+		)
+		(property "Value" "+3.3V"
+			(at 45.72 73.66 0)
+			(show_name no)
+			(do_not_autoplace no)
+			(effects
+				(font
+					(size 1.27 1.27)
+				)
+			)
+		)
+		(property "Footprint" ""
+			(at 45.72 78.74 0)
+			(hide yes)
+			(show_name no)
+			(do_not_autoplace no)
+			(effects
+				(font
+					(size 1.27 1.27)
+				)
+			)
+		)
+		(property "Datasheet" ""
+			(at 45.72 78.74 0)
+			(hide yes)
+			(show_name no)
+			(do_not_autoplace no)
+			(effects
+				(font
+					(size 1.27 1.27)
+				)
+			)
+		)
+		(property "Description" "Power symbol creates a global label with name \"+3.3V\""
+			(at 45.72 78.74 0)
+			(hide yes)
+			(show_name no)
+			(do_not_autoplace no)
+			(effects
+				(font
+					(size 1.27 1.27)
+				)
+			)
+		)
+		(pin "1"
+		)
+		(instances
+			(project "OpenAIO-Base"
+				(path "/fb88b6f9-ee39-4640-a9d4-04a17ceeac64/067dfe4f-0feb-4fee-b449-2d51932eecf1"
+					(reference "#PWR0289")
+					(unit 1)
+				)

Commit message: Schematic readability: TP texts, C19/C107, C26, title blocks (FB5 item 6, V9-V11/M6)
- TestPoint values ('TestPoint') hidden on all sheets: the stacked TP16/TP17
  (root), TP24/TP25 and TP18/TP19/TP26/TP27 (RP2354A) texts no longer overlap.
- C19 reference/value moved left of the part (no longer printed over C107).
- C26 Description field hidden.
- Title blocks: rev r2, date 2026-10 (title added where missing) on the root,
  RP2354A, Power, IMU, OSD, Pads, ESC channel and Core interface sheets.
Edited with kicad-skip, re-saved with `kicad-cli sch upgrade --force` so the
diff stays minimal. Not done: rx_esp32c3_sx1281 and fc_blackbox title blocks
(they carry other projects' instances, OpenRX-Lite / BLACKBOX, and the headless
re-save renumbers their references); TP10 outside the frame (moving it would
detach its wire); N4 SPI0 label lift (label position is the connection point);
M7 net naming (+4v5 / +3.3V vs +3V3) left as is, it touches the LGA spec.
ERC 31 errors (unchanged).

Co-Authored-By: Claude Opus 5.5 <noreply@anthropic.com>
Claude-Session: https://claude.ai/code/session_01KTp3FLjVXfXdWrkmr6af7d
Other:
- title: (none) -> IMU
Changed lines of the file:
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@@
 	(generator_version "10.0")
 	(paper "A5")
+	(title_block
+		(title "IMU")
+		(date "2026-10")
+		(rev "r2")
+	)
 	(polyline
 		(pts

Commit message: One board: merge Base and Core onto the OpenAIO-Whoop 8L HDI stackup
- hardware/OpenAIO.kicad_pcb: the routed Base and Core layouts of 8fa8d7b
  side by side in one board, all routing kept (Core promoted to 8 layers
  before the append so no Base layer was dropped). J90/J91 LGA deleted;
  their 46 nets are now direct links (51 unconnected, listed in
  research/ROUTING.md). Stackup and board setup from OpenAIO-Whoop:
  8L HDI 1+6+1, 0.997 mm, 1 oz all layers, microvia 0.25/0.10,
  buried 0.33/0.15. Base DRC severities and exclusions kept.
- hardware/OpenAIO.kicad_dru: canonical block, Whoop HDI via rules,
  Base/Core rules that still apply; LGA, 2 oz and 1.6 mm via rules gone.
- Schematic: core_interface sheet removed; DPS368 baro U28 on I2C0;
  review fixes (U3 HF cap C116, RP2354 caps C117/C118, buzzer flyback D10,
  SD card on +3.3V, D9 on +4v5, FLASH_CS -> SD_CS, PWR_FLAGs, U7 pin
  names, ESC cap pin types, L4 LCSC). ERC 32 -> 0 errors.
- Libraries project-local: every footprint, 3D model and symbol in lib;
  OPENDRONE_LIB aliases removed from the lib tables.
- Two-board projects, multiboard config and LGA tools removed; Whoop
  board tools added in hardware/tools.
- Docs: README, AGENTS.md, research/ROUTING.md (hand-over),
  SCHEMATIC-REVIEW-2026-10-15.md, Betaflight target baro.

DRC: 38 errors (25 dangling LGA escape vias, 13 Core leftovers listed),
51 unconnected (the Base-Core links), 0 net or value parity issues.

Co-Authored-By: Claude Opus 5.5 <noreply@anthropic.com>
Parts:
- C29, C30: footprint Capacitor_SMD:C_0201_0603Metric -> lib:C_0201_0603Metric
- R25: footprint Resistor_SMD:R_0201_0603Metric -> lib:R_0201_0603Metric
Changed lines of the file:
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@@
 			)
 		)
-		(property "Footprint" "Resistor_SMD:R_0201_0603Metric"
+		(property "Footprint" "lib:R_0201_0603Metric"
 			(at 107.95 80.518 90)
 			(hide yes)
@@
 	)
 	(symbol
-		(lib_name "+3.3V_1")
-		(lib_id "power:+3.3V")
+		(lib_id "lib:+3.3V_1")
 		(at 83.82 43.18 0)
 		(unit 1)
@@
 			)
 		)
-		(property "Footprint" "Capacitor_SMD:C_0201_0603Metric"
+		(property "Footprint" "lib:C_0201_0603Metric"
 			(at 63.1952 50.8 0)
 			(hide yes)
@@
 	)
 	(symbol
-		(lib_name "+3.3V_1")
-		(lib_id "power:+3.3V")
+		(lib_id "lib:+3.3V_1")
 		(at 45.72 78.74 0)
 		(unit 1)
@@
 			)
 		)
-		(property "Footprint" "Capacitor_SMD:C_0201_0603Metric"
+		(property "Footprint" "lib:C_0201_0603Metric"
 			(at 84.7852 50.8 0)
 			(hide yes)

Commit message: One board from the owner's 2026-08-22 Base and Core, BMP580 baro (#26)
The board is rebuilt from d81e559 (the hand-routed Base recovered from KiCad
local history and the hand-routed Core of 1fe3d21) plus the always-on +10V of
9aba717, instead of the agent-reworked 8fa8d7b. Both layouts sit side by side
in hardware/OpenAIO.kicad_pcb with all routing kept (2513 tracks, 1577 vias),
on the OpenAIO-Whoop 8L HDI stackup.

- Schematic: Core_Interface (J90/J91 LGA) removed; U26 BMP580 + C107/C108 on
  I2C0 at 0x47 (Betaflight BMP5xx default). Netlist otherwise identical to
  9aba717; ERC 31 errors, the 9aba717 baseline.
- Board: Base netclasses and severities; rule area "Core layout" keeps the
  Core's 0.09 line standard. DRC: 3 errors (USB1 peg), 37 unconnected (links).
- lib.pretty footprints replaced by the board instances; BMP580 imported with
  easyeda2kicad (LCSC C22391138).
- Not carried from 8fa8d7b: TXU0101 LED-strip buffer, +3V3_ESC, SWD pads,
  DFM edits; firmware ISSUES I2/I3 reopened.
- Docs: README pinout re-measured, AGENTS.md, research/ROUTING.md, Betaflight
  target USE_BARO_BMP580.

Co-authored-by: Stan <stan@openaio.local>
Co-authored-by: Claude Opus 5.5 <noreply@anthropic.com>
Connections:
- net +3.3V: no longer U8.2 (SDx/AH1/Qvar1), U8.3 (SCx/AH2/Qvar2)
- net GND: now also U8.2 (SDx/AH1/Qvar1), U8.3 (SCx/AH2/Qvar2)
Other:
- title: IMU -> (none)
Changed lines of the file:
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@@
 	(generator_version "10.0")
 	(paper "A5")
-	(title_block
-		(title "IMU")
-		(date "2026-10")
-		(rev "r2")
-	)
 	(polyline
 		(pts
@@
 		(color 0 0 0 0)
 	)
+	(junction
+		(at 45.72 81.28)
+		(diameter 0)
+		(color 0 0 0 0)
+	)
 	(no_connect
 		(at 93.98 78.74)
@@
 		(pts
 			(xy 73.66 57.15) (xy 73.66 43.18)
+		)
+		(stroke
+			(width 0)
+			(type default)
+		)
+	)
+	(wire
+		(pts
+			(xy 45.72 92.71) (xy 45.72 81.28)
 		)
 		(stroke
@@
 	(symbol
 		(lib_id "power:GND")
+		(at 45.72 92.71 0)
+		(unit 1)
+		(body_style 1)
+		(exclude_from_sim no)
+		(in_bom yes)
+		(on_board yes)
+		(in_pos_files yes)
+		(dnp no)
+		(fields_autoplaced yes)
+		(property "Reference" "#PWR076"
+			(at 45.72 99.06 0)
+			(hide yes)
+			(show_name no)
+			(do_not_autoplace no)
+			(effects
+				(font
+					(size 1.27 1.27)
+				)
+			)
+		)
+		(property "Value" "GND"
+			(at 45.72 97.79 0)
+			(show_name no)
+			(do_not_autoplace no)
+			(effects
+				(font
+					(size 1.27 1.27)
+				)
+			)
+		)
+		(property "Footprint" ""
+			(at 45.72 92.71 0)
+			(hide yes)
+			(show_name no)
+			(do_not_autoplace no)
+			(effects
+				(font
+					(size 1.27 1.27)
+				)
+			)
+		)
+		(property "Datasheet" ""
+			(at 45.72 92.71 0)
+			(hide yes)
+			(show_name no)
+			(do_not_autoplace no)
+			(effects
+				(font
+					(size 1.27 1.27)
+				)
+			)
+		)
+		(property "Description" "Power symbol creates a global label with name \"GND\" , ground"
+			(at 45.72 92.71 0)
+			(hide yes)
+			(show_name no)
+			(do_not_autoplace no)
+			(effects
+				(font
+					(size 1.27 1.27)
+				)
+			)
+		)
+		(pin "1"
+		)
+		(instances
+			(project "OpenAIO-Base"
+				(path "/fb88b6f9-ee39-4640-a9d4-04a17ceeac64/067dfe4f-0feb-4fee-b449-2d51932eecf1"
+					(reference "#PWR076")
+					(unit 1)
+				)
+			)
+		)
+	)
+	(symbol
+		(lib_id "power:GND")
 		(at 83.82 50.8 0)
 		(unit 1)
@@
 					(unit 1)
 				)
-			)
-		)
-	)
-	(symbol
-		(lib_id "lib:+3.3V_1")
-		(at 45.72 78.74 0)
-		(unit 1)
-		(body_style 1)
-		(exclude_from_sim no)
-		(in_bom yes)
-		(on_board yes)
-		(in_pos_files yes)
-		(dnp no)
-		(fields_autoplaced yes)
-		(property "Reference" "#PWR0289"
-			(at 45.72 82.55 0)
-			(hide yes)
-			(show_name no)
-			(do_not_autoplace no)
-			(effects
-				(font
-					(size 1.27 1.27)
-				)
-			)
-		)
-		(property "Value" "+3.3V"
-			(at 45.72 73.66 0)
-			(show_name no)
-			(do_not_autoplace no)
-			(effects
-				(font
-					(size 1.27 1.27)
-				)
-			)
-		)
-		(property "Footprint" ""
-			(at 45.72 78.74 0)
-			(hide yes)
-			(show_name no)
-			(do_not_autoplace no)
-			(effects
-				(font
-					(size 1.27 1.27)
-				)
-			)
-		)
-		(property "Datasheet" ""
-			(at 45.72 78.74 0)
-			(hide yes)
-			(show_name no)
-			(do_not_autoplace no)
-			(effects
-				(font
-					(size 1.27 1.27)
-				)
-			)
-		)
-		(property "Description" "Power symbol creates a global label with name \"+3.3V\""
-			(at 45.72 78.74 0)
-			(hide yes)
-			(show_name no)
-			(do_not_autoplace no)
-			(effects
-				(font
-					(size 1.27 1.27)
-				)
-			)
-		)
-		(pin "1"
-		)
-		(instances
-			(project "OpenAIO-Base"
-				(path "/fb88b6f9-ee39-4640-a9d4-04a17ceeac64/067dfe4f-0feb-4fee-b449-2d51932eecf1"
-					(reference "#PWR0289")
-					(unit 1)
-				)
