File: hardware/fc_imu.kicad_sch (KiCad schematic)
At the start: 4 parts, among them U8 BMI270

Commit message: Library: every symbol, footprint and 3D model project-local (#28)
* Owner: board cleanup, Core placed on the board

Co-Authored-By: Claude Opus 5.5 <noreply@anthropic.com>

* Library: every symbol, footprint and 3D model project-local

- 3D models: 275 board model paths and 28 lib.pretty footprints pointed at
  KiCad's stock install or at ${OPENDRONE_LIB} (which this machine's KiCad sets
  to a path that does not exist, so 9 models were missing). All now resolve to
  ${KIPRJMOD}/lib.3dshapes; the three missing ones come from the repo's
  KiCad-Library submodule. .wrl replaced by the .step sibling where one exists.
- Symbols: the 14 stock symbols (Device, power, Connector, Connector_Generic,
  MCU_Espressif) copied into lib.kicad_sym from the schematic's own cache and
  relinked as lib:. Four lib symbols refreshed from the schematic (they still
  held the 8fa8d7b copies).
- Pruned: 11 unused footprints, 7 unused symbols, unreferenced model files.
- tools/localise_models.py and tools/localise_symbols.py keep it that way.
- Checks: board diff is model lines only; netlist identical; ERC 31 errors as
  before, lib_symbol_mismatch 9 -> 0.

Co-Authored-By: Claude Opus 5.5 <noreply@anthropic.com>

---------

Co-authored-by: Stan <stan@openaio.local>
Co-authored-by: Claude Opus 5.5 <noreply@anthropic.com>
Parts:
- C29, C30: symbol Device:C -> lib:C
- R25: symbol Device:R -> lib:R
Changed lines of the file:
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@@
 	)
 	(symbol
-		(lib_id "Device:R")
+		(lib_id "lib:R")
 		(at 107.95 78.74 90)
 		(unit 1)
@@
 	)
 	(symbol
-		(lib_id "power:+3.3V")
+		(lib_id "lib:+3.3V")
 		(at 111.76 78.74 270)
 		(unit 1)
@@
 	)
 	(symbol
-		(lib_id "power:GND")
+		(lib_id "lib:GND")
 		(at 45.72 92.71 0)
 		(unit 1)
@@
 	)
 	(symbol
-		(lib_id "power:GND")
+		(lib_id "lib:GND")
 		(at 83.82 50.8 0)
 		(unit 1)
@@
 	)
 	(symbol
-		(lib_id "Device:C")
+		(lib_id "lib:C")
 		(at 62.23 46.99 0)
 		(unit 1)
@@
 	)
 	(symbol
-		(lib_id "power:+3.3V")
+		(lib_id "lib:+3.3V")
 		(at 62.23 43.18 0)
 		(unit 1)
@@
 	)
 	(symbol
-		(lib_id "power:GND")
+		(lib_id "lib:GND")
 		(at 62.23 50.8 0)
 		(unit 1)
@@
 	)
 	(symbol
-		(lib_id "power:GND")
+		(lib_id "lib:GND")
 		(at 72.39 92.71 0)
 		(unit 1)
@@
 	)
 	(symbol
-		(lib_id "Device:C")
+		(lib_id "lib:C")
 		(at 83.82 46.99 0)
 		(unit 1)
