File: hardware/fc_osd.kicad_sch (KiCad schematic)
At the start: 17 parts, among them U10 COS8051SOT, U11 TLV7031DPWR, U9 SN74LVC1G3157DTBR

Commit message: Owner rules: no component silk, pad labels and values, no wordmark text, MPN + maker on every BOM line
The owner rules adopted in PLAN.md (pcb-agent-commons, 2026-10-06), applied
where they are local edits:

- No component silkscreen. J91's reference was the only visible one (Core
  B.Silkscreen, under the LGA) and is hidden. Footprint silk graphics removed
  per instance: Base 234, Core 72. Kept: connector outlines and pin-1 marks
  (USB1, U12 SH-6, Card1, JP1) and the LGA pin-1 marks (J90, J91). Base
  lib_footprint_mismatch warnings 31 -> 40 as a result.
- Solder-pad labels: Core J53 (GND) had none, now "gnd" in the style of J52's
  label. The SH-6 per-pin labels ("10v gnd T0", "R0 gnd R1") become the port
  name "DJI" (connectors: name and pin-1 mark only). Core J48-J51 have no room:
  0.5 mm to J44 above, 0.93 mm to the board edge below. CIRCUIT_REVIEW 8.3
  moves them off the LGA in R2, so their labels go with that move.
- Pad values: all 40 solder-pad symbols said "5V". Each now carries its
  function (5V, GND, LED, BUZ+/BUZ-, 10V, 4V5, CAM, VTX, SCL, SDA, TX0/RX0,
  TX1/RX1, PIO_TX0/PIO_RX0; off-board J19 ADC2, J22 GND, J46/J47 NC).
- No "Drone" text: the "OpenDrone" wordmark on Core F.Silkscreen (9 filled
  polygons in two groups) is removed; a TODO for the incutec wordmark from the
  brand repo sits on User.Comments (not fabricated). No other such text on any
  copper, mask or silk layer of either board.
- BOM: lines missing manufacturer or MPN 41 -> 1. MPNs come from
  PARTS-USED.md by LCSC number. Manufacturers come from the catalogue symbol,
  this design's spelling for the same MPN family, or the committed datasheet
  (NSIC, Sofng, Jiangsu Changjing, Hirose). Still open: Rsense2
  ASR-S-3-0.2F (C695806), whose manufacturer nothing in the catalogue states.
  U24 (board outline) and TP9 (BOOT solder pad) are not parts: excluded from
  BOM and position files.
- 0201 default / minimal capacitance: respected in the circuit commit (C26
  stays 0201; no belt-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
Parts:
- R31, R32: MPN (none) -> RC0201FR-07510RL; Manufacturer (none) -> YAGEO
Changed lines of the file:
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@@
 			)
 		)
-		(property "MPN" ""
+		(property "MPN" "RC0201FR-07510RL"
 			(at -74.93 83.82 0)
 			(hide yes)
@@
 			)
 		)
-		(property "Manufacturer" ""
+		(property "Manufacturer" "YAGEO"
 			(at -74.93 83.82 0)
 			(hide yes)
@@
 			)
 		)
-		(property "MPN" ""
+		(property "MPN" "RC0201FR-07510RL"
 			(at 95.25 434.34 0)
 			(hide yes)
@@
 			)
 		)
-		(property "Manufacturer" ""
+		(property "Manufacturer" "YAGEO"
 			(at 95.25 434.34 0)
 			(hide yes)

Commit message: Schematic readability: TP texts, C19/C107, C26, title blocks (FB5 item 6, V9-V11/M6)
- TestPoint values ('TestPoint') hidden on all sheets: the stacked TP16/TP17
  (root), TP24/TP25 and TP18/TP19/TP26/TP27 (RP2354A) texts no longer overlap.
- C19 reference/value moved left of the part (no longer printed over C107).
- C26 Description field hidden.
- Title blocks: rev r2, date 2026-10 (title added where missing) on the root,
  RP2354A, Power, IMU, OSD, Pads, ESC channel and Core interface sheets.
Edited with kicad-skip, re-saved with `kicad-cli sch upgrade --force` so the
diff stays minimal. Not done: rx_esp32c3_sx1281 and fc_blackbox title blocks
(they carry other projects' instances, OpenRX-Lite / BLACKBOX, and the headless
re-save renumbers their references); TP10 outside the frame (moving it would
detach its wire); N4 SPI0 label lift (label position is the connection point);
M7 net naming (+4v5 / +3.3V vs +3V3) left as is, it touches the LGA spec.
ERC 31 errors (unchanged).

Co-Authored-By: Claude Opus 5.5 <noreply@anthropic.com>
Claude-Session: https://claude.ai/code/session_01KTp3FLjVXfXdWrkmr6af7d
Other:
- title: (none) -> OSD
Changed lines of the file:
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@@
 	(generator_version "10.0")
 	(paper "A3")
+	(title_block
+		(title "OSD")
+		(date "2026-10")
+		(rev "r2")
+	)
 	(polyline
 		(pts

Commit message: One board: merge Base and Core onto the OpenAIO-Whoop 8L HDI stackup
- hardware/OpenAIO.kicad_pcb: the routed Base and Core layouts of 8fa8d7b
  side by side in one board, all routing kept (Core promoted to 8 layers
  before the append so no Base layer was dropped). J90/J91 LGA deleted;
  their 46 nets are now direct links (51 unconnected, listed in
  research/ROUTING.md). Stackup and board setup from OpenAIO-Whoop:
  8L HDI 1+6+1, 0.997 mm, 1 oz all layers, microvia 0.25/0.10,
  buried 0.33/0.15. Base DRC severities and exclusions kept.
- hardware/OpenAIO.kicad_dru: canonical block, Whoop HDI via rules,
  Base/Core rules that still apply; LGA, 2 oz and 1.6 mm via rules gone.
- Schematic: core_interface sheet removed; DPS368 baro U28 on I2C0;
  review fixes (U3 HF cap C116, RP2354 caps C117/C118, buzzer flyback D10,
  SD card on +3.3V, D9 on +4v5, FLASH_CS -> SD_CS, PWR_FLAGs, U7 pin
  names, ESC cap pin types, L4 LCSC). ERC 32 -> 0 errors.
- Libraries project-local: every footprint, 3D model and symbol in lib;
  OPENDRONE_LIB aliases removed from the lib tables.
- Two-board projects, multiboard config and LGA tools removed; Whoop
  board tools added in hardware/tools.
- Docs: README, AGENTS.md, research/ROUTING.md (hand-over),
  SCHEMATIC-REVIEW-2026-10-15.md, Betaflight target baro.

DRC: 38 errors (25 dangling LGA escape vias, 13 Core leftovers listed),
51 unconnected (the Base-Core links), 0 net or value parity issues.

Co-Authored-By: Claude Opus 5.5 <noreply@anthropic.com>
Parts:
- C31, C32, C34, C35: footprint Capacitor_SMD:C_0201_0603Metric -> lib:C_0201_0603Metric
- C33: footprint Capacitor_SMD:C_0402_1005Metric -> lib:C_0402_1005Metric
- R26, R27, R28, R29, R30, R31, R32, R33: footprint Resistor_SMD:R_0201_0603Metric -> lib:R_0201_0603Metric
Changed lines of the file:
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@@
 			)
 		)
-		(property "Footprint" "Capacitor_SMD:C_0201_0603Metric"
+		(property "Footprint" "lib:C_0201_0603Metric"
 			(at 138.1252 119.38 0)
 			(hide yes)
@@
 			)
 		)
-		(property "Footprint" "Resistor_SMD:R_0201_0603Metric"
+		(property "Footprint" "lib:R_0201_0603Metric"
 			(at 97.79 169.418 90)
 			(hide yes)
@@
 			)
 		)
-		(property "Footprint" "Resistor_SMD:R_0201_0603Metric"
+		(property "Footprint" "lib:R_0201_0603Metric"
 			(at 176.022 187.96 90)
 			(hide yes)
@@
 			)
 		)
-		(property "Footprint" "Resistor_SMD:R_0201_0603Metric"
+		(property "Footprint" "lib:R_0201_0603Metric"
 			(at 110.998 161.29 90)
 			(hide yes)
@@
 			)
 		)
-		(property "Footprint" "Capacitor_SMD:C_0201_0603Metric"
+		(property "Footprint" "lib:C_0201_0603Metric"
 			(at 183.8452 146.05 0)
 			(hide yes)
@@
 			)
 		)
-		(property "Footprint" "Resistor_SMD:R_0201_0603Metric"
+		(property "Footprint" "lib:R_0201_0603Metric"
 			(at 208.28 166.878 90)
 			(hide yes)
@@
 			)
 		)
-		(property "Footprint" "Capacitor_SMD:C_0201_0603Metric"
+		(property "Footprint" "lib:C_0201_0603Metric"
 			(at 143.2052 146.05 0)
 			(hide yes)
@@
 			)
 		)
-		(property "Footprint" "Resistor_SMD:R_0201_0603Metric"
+		(property "Footprint" "lib:R_0201_0603Metric"
 			(at 110.998 173.99 90)
 			(hide yes)
@@
 			)
 		)
-		(property "Footprint" "Resistor_SMD:R_0201_0603Metric"
+		(property "Footprint" "lib:R_0201_0603Metric"
 			(at 96.012 115.57 90)
 			(hide yes)
@@
 			)
 		)
-		(property "Footprint" "Capacitor_SMD:C_0402_1005Metric"
+		(property "Footprint" "lib:C_0402_1005Metric"
 			(at 163.83 108.2548 0)
 			(hide yes)
@@
 			)
 		)
-		(property "Footprint" "Capacitor_SMD:C_0201_0603Metric"
+		(property "Footprint" "lib:C_0201_0603Metric"
 			(at 219.4052 92.71 0)
 			(hide yes)
@@
 			)
 		)
-		(property "Footprint" "Resistor_SMD:R_0201_0603Metric"
+		(property "Footprint" "lib:R_0201_0603Metric"
 			(at 129.54 107.442 90)
 			(hide yes)
@@
 			)
 		)
-		(property "Footprint" "Resistor_SMD:R_0201_0603Metric"
+		(property "Footprint" "lib:R_0201_0603Metric"
 			(at 199.39 183.388 90)
 			(hide yes)

Commit message: One board from the owner's 2026-08-22 Base and Core, BMP580 baro (#26)
The board is rebuilt from d81e559 (the hand-routed Base recovered from KiCad
local history and the hand-routed Core of 1fe3d21) plus the always-on +10V of
9aba717, instead of the agent-reworked 8fa8d7b. Both layouts sit side by side
in hardware/OpenAIO.kicad_pcb with all routing kept (2513 tracks, 1577 vias),
on the OpenAIO-Whoop 8L HDI stackup.

- Schematic: Core_Interface (J90/J91 LGA) removed; U26 BMP580 + C107/C108 on
  I2C0 at 0x47 (Betaflight BMP5xx default). Netlist otherwise identical to
  9aba717; ERC 31 errors, the 9aba717 baseline.
- Board: Base netclasses and severities; rule area "Core layout" keeps the
  Core's 0.09 line standard. DRC: 3 errors (USB1 peg), 37 unconnected (links).
- lib.pretty footprints replaced by the board instances; BMP580 imported with
  easyeda2kicad (LCSC C22391138).
- Not carried from 8fa8d7b: TXU0101 LED-strip buffer, +3V3_ESC, SWD pads,
  DFM edits; firmware ISSUES I2/I3 reopened.
- Docs: README pinout re-measured, AGENTS.md, research/ROUTING.md, Betaflight
  target USE_BARO_BMP580.

Co-authored-by: Stan <stan@openaio.local>
Co-authored-by: Claude Opus 5.5 <noreply@anthropic.com>
Parts:
- R31, R32: MPN RC0201FR-07510RL -> (none); Manufacturer YAGEO -> (none)
Other:
- title: OSD -> (none)
Changed lines of the file:
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@@
 	(generator_version "10.0")
 	(paper "A3")
-	(title_block
-		(title "OSD")
-		(date "2026-10")
-		(rev "r2")
-	)
 	(polyline
 		(pts
@@
 			)
 		)
-		(property "MPN" "RC0201FR-07510RL"
+		(property "MPN" ""
 			(at -74.93 83.82 0)
 			(hide yes)
@@
 			)
 		)
-		(property "Manufacturer" "YAGEO"
+		(property "Manufacturer" ""
 			(at -74.93 83.82 0)
 			(hide yes)
@@
 			)
 		)
-		(property "MPN" "RC0201FR-07510RL"
+		(property "MPN" ""
 			(at 95.25 434.34 0)
 			(hide yes)
@@
 			)
 		)
-		(property "Manufacturer" "YAGEO"
+		(property "Manufacturer" ""
 			(at 95.25 434.34 0)
 			(hide yes)
