File: hardware/OpenAIO.kicad_pcb (KiCad board)
At the start: 6 copper layers, 35 x 35 mm, 325 parts, among them J21 5V, J23 5V, J25 5V, J26 5V, J28 5V, J29 5V, J30 5V, J32 5V, J33 5V, J34 5V, J35 5V, J36 5V, J37 5V, J38 5V, J39 5V, J42 5V, J43 5V, J44 5V, J45 5V, J48 5V, J49 5V, J50 5V, J51 5V, J90 Core_LGA, J91 Core_LGA, Q1 AP1606, Q10 DOY180N03T, Q11 DOY180N03T, Q12 DOY180N03T, Q13 DOY180N03T, Q14 DOY180N03T, Q15 DOY180N03T, Q16 DOY180N03T, Q17 DOY180N03T, Q18 DOY180N03T, Q19 DOY180N03T, Q2 AP1606, Q20 DOY180N03T, Q21 DOY180N03T, Q22 DOY180N03T, Q23 DOY180N03T, Q24 DOY180N03T, Q25 DOY180N03T, Q26 DOY180N03T, Q3 DOY180N03T, Q4 DOY180N03T, Q5 DOY180N03T, Q6 DOY180N03T, Q7 DOY180N03T, Q8 DOY180N03T, Q9 DOY180N03T, U1 TS2306A 240GF MSM 9_C2976675, U10 COS8051SOT, U11 TLV7031DPWR, U12 SM06B-SRSS-TB(LF)(SN), U13 AT32F421G8U7, U14 NSG2065Q, U15 AT32F421G8U7, U16 NSG2065Q, U17 AT32F421G8U7, U18 NSG2065Q, U19 AT32F421G8U7, U2 RP2354A, U20 NSG2065Q, U21 SX1281IMLTRT, U22 ESP32-C3, U23 TLV75533PDQNR, U24 AIO_outline, U25 INA186A3IDCKR, U3 LMR51430YFDDCR, U4 LMR51430YFDDCR, U6 LP5912-1.8DRVR, U7 LP5912-3.3DRVR, U8 BMI270, U9 SN74LVC1G3157DTBR, X1 XTM25012000JT00351001, X2 CJ17-400001010B20

Commit message: OpenAIO: Core outline from User.2 to Edge.Cuts, J90/J91 re-placed with nets, Core rule area, derived boards refreshed
tools/core_outline.py moves the closed User.2 contour of the Core island to
Edge.Cuts. J90 sits in the free area of the Base top (78.9, 62.0), J91 inside
the Core outline (114.1, 53.55) on B.Cu; lga_place.py now assigns pad nets
from the pin table. Rule area Core redrawn from the new outline; split re-run,
J90 carries the new Core STEP and 23.1 x 20.2 mm shadow.
Parts:
- removed J36: 5V, lib:small_pad
- added C105: C, Capacitor_SMD:C_1206_3216Metric, F.Cu at (84.4, 50.6)
- added C106: C, Capacitor_SMD:C_1206_3216Metric, F.Cu at (78.9, 50.6)
- added J15: 5V, lib:small_pad, F.Cu at (61.9, 44.7)
- added J16: 5V, lib:small_pad, F.Cu at (59.1, 74.4)
- added J17: 5V, lib:small_pad, F.Cu at (60.2, 45.8)
- added J18: 5V, lib:small_pad, F.Cu at (60.2, 76.1)
- added J20: 5V, lib:small_pad, F.Cu at (59.1, 47.5)
- added J24: 5V, lib:small_pad, F.Cu at (91.7, 47.5)
- added J27: 5V, lib:small_pad, F.Cu at (90.6, 45.8)
- added J31: 5V, lib:small_pad, F.Cu at (88.9, 44.7)
- added J40: 5V, lib:small_pad, F.Cu at (108.2, 44.9)
- added J41: 5V, lib:small_pad, F.Cu at (106.2, 44.9)
- added J52: 5V, lib:small_pad, F.Cu at (118.8, 48.6)
- added J53: 5V, lib:small_pad, F.Cu at (118.8, 50.6)
- added J54: 5V, lib:small_pad, F.Cu at (118.8, 46.6)
- added J55: 5V, lib:small_pad, F.Cu at (118.8, 44.6)
- added TP9: BOOT, OpenRX-Shared:SolderPad_1.2x2.0mm, B.Cu at (79.7, 67.7)
- J29, J33: moved to B.Cu
- moved J21 56.7 mm to (61.9, 77.2), turned to 45 degrees
- moved J39 29.9 mm to (104.2, 44.9), turned to -90 degrees
- moved J29 29.8 mm to (90.6, 61.5)
- moved J33 29.7 mm to (90.6, 63.5)
- moved J32 29.6 mm to (91.7, 74.3), turned to 135 degrees
- moved J25 29.3 mm to (88.9, 77.1), turned to 135 degrees
- moved J34 26.4 mm to (114.2, 44.9), turned to 90 degrees
- moved J28 26.3 mm to (90.6, 76.0), turned to 135 degrees
- moved J26 26.1 mm to (112.2, 44.9), turned to 90 degrees
- moved J23 21.5 mm to (110.2, 44.9), turned to 90 degrees
- moved J35 20.6 mm to (124.8, 53.2)
- moved J43 20.1 mm to (121.0, 53.2)
- moved J30 18.3 mm to (116.2, 44.9), turned to 90 degrees
- moved J44 16.8 mm to (121.0, 59.2), turned to 180 degrees
- moved J51 16.2 mm to (115.2, 61.5), turned to -90 degrees
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Connections:
- Card1 pad 2: /Blackbox/FLASH_CS -> FLASH_CS
- Card1 pad 3: /Blackbox/SPI0.MOSI -> SPI0.MOSI
- Card1 pad 5: /Blackbox/SPI0.SCK -> SPI0.SCK
- Card1 pad 7: /Blackbox/SPI0.MISO -> SPI0.MISO
- J48 pad 1: /Pads/UART0_RX -> UART0_RX
- J49 pad 1: /Pads/UART0_TX -> UART0_TX
- J90 pad 1: (no net) -> GND
- J90 pad 10: (no net) -> +3.3V
- J90 pad 11: (no net) -> +3.3V
- J90 pad 12: (no net) -> +4v5
- J90 pad 13: (no net) -> GND
- J90 pad 14: (no net) -> 10V_ENABLE
- J90 pad 15: (no net) -> CURR
- J90 pad 16: (no net) -> GND
- J90 pad 17: (no net) -> GND
- J90 pad 18: (no net) -> USB_D+
- J90 pad 19: (no net) -> USB_D-
- J90 pad 2: (no net) -> +BATT
- J90 pad 20: (no net) -> GND
- J90 pad 21: (no net) -> MOTOR1
- J90 pad 22: (no net) -> MOTOR2
- J90 pad 23: (no net) -> MOTOR3
- J90 pad 24: (no net) -> MOTOR4
- J90 pad 25: (no net) -> UART0_TX
- J90 pad 26: (no net) -> UART0_RX
- J90 pad 27: (no net) -> UART1_TX
- J90 pad 28: (no net) -> UART1_RX
- J90 pad 29: (no net) -> SPI0.SCK
- J90 pad 3: (no net) -> GND
- J90 pad 30: (no net) -> SPI0.MOSI
- J90 pad 31: (no net) -> SPI0.MISO
- J90 pad 32: (no net) -> FLASH_CS
- J90 pad 4: (no net) -> +5V
- J90 pad 5: (no net) -> +5V
- J90 pad 6: (no net) -> GND
- J90 pad 7: (no net) -> +10V
- J90 pad 8: (no net) -> +10V
- J90 pad 9: (no net) -> GND
- J91 pad 1: (no net) -> GND
- J91 pad 10: (no net) -> +3.3V
- J91 pad 11: (no net) -> +3.3V
- J91 pad 12: (no net) -> +4v5
- J91 pad 13: (no net) -> GND
- J91 pad 14: (no net) -> 10V_ENABLE
- J91 pad 15: (no net) -> CURR
- J91 pad 16: (no net) -> GND
- J91 pad 17: (no net) -> GND
- J91 pad 18: (no net) -> USB_D+
- J91 pad 19: (no net) -> USB_D-
- J91 pad 2: (no net) -> +BATT
- J91 pad 20: (no net) -> GND
- J91 pad 21: (no net) -> MOTOR1
- J91 pad 22: (no net) -> MOTOR2
- J91 pad 23: (no net) -> MOTOR3
- J91 pad 24: (no net) -> MOTOR4
- J91 pad 25: (no net) -> UART0_TX
- J91 pad 26: (no net) -> UART0_RX
- J91 pad 27: (no net) -> UART1_TX
- J91 pad 28: (no net) -> UART1_RX
- J91 pad 29: (no net) -> SPI0.SCK
- J91 pad 3: (no net) -> GND
- J91 pad 30: (no net) -> SPI0.MOSI
- J91 pad 31: (no net) -> SPI0.MISO
- J91 pad 32: (no net) -> FLASH_CS
- J91 pad 4: (no net) -> +5V
- J91 pad 5: (no net) -> +5V
- J91 pad 6: (no net) -> GND
- J91 pad 7: (no net) -> +10V
- J91 pad 8: (no net) -> +10V
- J91 pad 9: (no net) -> GND
- R34 pad 2: /Blackbox/FLASH_CS -> FLASH_CS
- R39 pad 1: /ESC1/dshot -> MOTOR1
- R5 pad 1: /RP2354A/ESC_CURRENT -> CURR
- R58 pad 1: /ESC2/dshot -> MOTOR2
- R77 pad 1: /ESC3/dshot -> MOTOR3
- R8 pad 1: /RP2354A/D- -> USB_D-
- R9 pad 2: /RP2354A/D+ -> USB_D+
- R96 pad 1: /ESC4/dshot -> MOTOR4
- U12 pad 3: /Pads/UART0_TX -> UART0_TX
- U12 pad 4: /Pads/UART0_RX -> UART0_RX
- U2 pad 10: /RP2354A/UART1_RX -> UART1_RX
- U2 pad 2: /Pads/UART0_TX -> UART0_TX
- U2 pad 29: /Blackbox/SPI0.SCK -> SPI0.SCK
- U2 pad 3: /Pads/UART0_RX -> UART0_RX
- U2 pad 31: /Blackbox/SPI0.MOSI -> SPI0.MOSI
- U2 pad 32: /Blackbox/SPI0.MISO -> SPI0.MISO
- U2 pad 33: /Blackbox/FLASH_CS -> FLASH_CS
- U2 pad 34: /ESC4/dshot -> MOTOR4
- U2 pad 35: /ESC3/dshot -> MOTOR3
- U2 pad 36: /ESC2/dshot -> MOTOR2
- U2 pad 37: /ESC1/dshot -> MOTOR1
- U2 pad 41: /Power/10V_ENABLE -> 10V_ENABLE
- U2 pad 9: /RP2354A/UART1_TX -> UART1_TX
- U22 pad 27: /RP2354A/UART1_TX -> UART1_TX
- U22 pad 28: /RP2354A/UART1_RX -> UART1_RX
- U25 pad 6: /CURR -> CURR
- U3 pad 5: /Power/10V_ENABLE -> 10V_ENABLE
- USB1 pad A6: /RP2354A/D+ -> USB_D+
- USB1 pad A7: /RP2354A/D- -> USB_D-
- USB1 pad B6: /RP2354A/D+ -> USB_D+
- USB1 pad B7: /RP2354A/D- -> USB_D-
Routing:
- net USB_D+: track 0.00 -> 4.29 mm
- net /RP2354A/D+: track 4.29 -> 0.00 mm
- net USB_D-: track 0.00 -> 2.86 mm
- net /RP2354A/D-: track 2.86 -> 0.00 mm, vias 2 -> 0
- net /OSD/OSD_LVL: track 3.05 -> 0.65 mm
- net 10V_ENABLE: track 0.00 -> 1.91 mm
- net /Power/10V_ENABLE: track 1.91 -> 0.00 mm, vias 1 -> 0
- net +3.3V: track 3.57 -> 2.43 mm, vias 1 -> 0
- net Net-(USB1-CC2): vias 1 -> 0
- net Net-(USB1-CC1): vias 1 -> 0
- net Net-(U4-SW): vias 1 -> 0
- net Net-(U3-SW): vias 1 -> 0
- net Net-(Q9-G): vias 2 -> 0
- net Net-(Q8-G): vias 2 -> 0
- net Net-(Q7-G): vias 2 -> 0
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Other:
- board text added: "+"
- board text added: "-"
