File: hardware/OpenAIO-Base.kicad_pcb (KiCad board)
At the start: 6 copper layers, 35 x 35 mm, 254 parts, among them J15 5V, J16 5V, J17 5V, J18 5V, J20 5V, J21 5V, J24 5V, J25 5V, J27 5V, J28 5V, J29 5V, J31 5V, J32 5V, J33 5V, J90 Core_LGA, Q10 DOY180N03T, Q11 DOY180N03T, Q12 DOY180N03T, Q13 DOY180N03T, Q14 DOY180N03T, Q15 DOY180N03T, Q16 DOY180N03T, Q17 DOY180N03T, Q18 DOY180N03T, Q19 DOY180N03T, Q20 DOY180N03T, Q21 DOY180N03T, Q22 DOY180N03T, Q23 DOY180N03T, Q24 DOY180N03T, Q25 DOY180N03T, Q26 DOY180N03T, Q3 DOY180N03T, Q4 DOY180N03T, Q5 DOY180N03T, Q6 DOY180N03T, Q7 DOY180N03T, Q8 DOY180N03T, Q9 DOY180N03T, U12 SM06B-SRSS-TB(LF)(SN), U13 AT32F421G8U7, U14 NSG2065Q, U15 AT32F421G8U7, U16 NSG2065Q, U17 AT32F421G8U7, U18 NSG2065Q, U19 AT32F421G8U7, U20 NSG2065Q, U21 SX1281IMLTRT, U22 ESP32-C3, U23 TLV75533PDQNR, U24 AIO_outline, U25 INA186A3IDCKR, U3 LMR51430YFDDCR, U4 LMR51430YFDDCR, U7 LP5912-3.3DRVR, X2 CJ17-400001010B20

Commit message: Base: routing progress (~60%), netclass clearances relaxed
VBAT/Phase/Power/RF clearance lowered toward the 0.09 line standard; the
2 oz outer rule in the DRU still enforces 0.16 on F/B.Cu. Schematic sheets
resaved by eeschema, no circuit change.
Parts:
- removed AE1: 47948-0001, OpenRX-Shared:ANT-SMD_47948-0001
- added JP1: U.FL-R-SMT-1(80), OpenDrone:RF-SMD_FRF05002-JSS103M, F.Cu at (91.1, 69.3)
- moved C83 0.48 mm to (83.4, 74.2), turned to 0 degrees
- moved C80 0.47 mm to (83.4, 73.6), turned to 0 degrees
- moved OSC1 0.13 mm to (85.2, 74.6)
- turned C105 to 180 degrees
Connections:
- U12 pad 6: /Pads/U1RX -> UART1_RX
Routing:
- net +10V: track 15.8 -> 56.4 mm, vias 7 -> 13
- net GND: track 61.3 -> 100.6 mm, vias 231 -> 355
- net FLASH_CS: track 0.00 -> 23.6 mm, vias 0 -> 2
- net /1A: track 0.91 -> 22.7 mm, vias 2 -> 21
- net /4C: track 2.58 -> 24.3 mm, vias 2 -> 20
- net /1C: track 1.70 -> 23.3 mm, vias 2 -> 20
- net /2B: track 0.95 -> 22.1 mm, vias 1 -> 21
- net /3A: track 0.94 -> 21.3 mm, vias 2 -> 21
- net /2A: track 0.90 -> 20.9 mm, vias 2 -> 21
- net /1B: track 0.85 -> 19.3 mm, vias 2 -> 21
- net SPI0.MOSI: track 0.00 -> 18.4 mm, vias 0 -> 2
- net /3B: track 1.56 -> 19.8 mm, vias 2 -> 20
- net /3C: track 2.39 -> 20.2 mm, vias 2 -> 21
- net +3V3: track 24.3 -> 41.8 mm, vias 7 -> 10
- net /4B: track 1.01 -> 18.0 mm, vias 3 -> 20
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- added copper zone on In5.Cu, net +10V
- added copper zone on In3.Cu, net +3V3
- added copper zone on B.Cu, net +BATT
- added copper zone on F.Cu, net +BATT
- added copper zone on In2.Cu, net +BATT
- added copper zone on In3.Cu, net +BATT
- added copper zone on B.Cu, net /1A
- added copper zone on F.Cu, net /1A
- added copper zone on In1.Cu, net /1A
- added copper zone on In2.Cu, net /1A
- added copper zone on In3.Cu, net /1A
- added copper zone on In4.Cu, net /1A
- added copper zone on B.Cu, net /1B
- added copper zone on F.Cu, net /1B
- added copper zone on In1.Cu, net /1B
- added copper zone on In2.Cu, net /1B
- added copper zone on In3.Cu, net /1B
- added copper zone on In4.Cu, net /1B
- added copper zone on B.Cu, net /1C
- added copper zone on F.Cu, net /1C
- added copper zone on In1.Cu, net /1C
- added copper zone on In2.Cu, net /1C
- added copper zone on In3.Cu, net /1C
- added copper zone on In4.Cu, net /1C
- added copper zone on B.Cu, net /2A
- added copper zone on F.Cu, net /2A
- added copper zone on In1.Cu, net /2A
- added copper zone on In2.Cu, net /2A
- added copper zone on In3.Cu, net /2A
- added copper zone on In4.Cu, net /2A
- added copper zone on B.Cu, net /2B
- added copper zone on F.Cu, net /2B
- added copper zone on In1.Cu, net /2B
- added copper zone on In2.Cu, net /2B
- added copper zone on In3.Cu, net /2B
- added copper zone on In4.Cu, net /2B
- added copper zone on B.Cu, net /2C
- added copper zone on F.Cu, net /2C
- added copper zone on In1.Cu, net /2C
- added copper zone on In2.Cu, net /2C
- added copper zone on In3.Cu, net /2C
- added copper zone on In4.Cu, net /2C
- added copper zone on B.Cu, net /3A
- added copper zone on F.Cu, net /3A
- added copper zone on In1.Cu, net /3A
- added copper zone on In2.Cu, net /3A
- added copper zone on In3.Cu, net /3A
- added copper zone on In4.Cu, net /3A
- added copper zone on B.Cu, net /3B
- added copper zone on F.Cu, net /3B
- added copper zone on In1.Cu, net /3B
- added copper zone on In2.Cu, net /3B
- added copper zone on In3.Cu, net /3B
- added copper zone on In4.Cu, net /3B
- added copper zone on B.Cu, net /3C
- added copper zone on F.Cu, net /3C
- added copper zone on In1.Cu, net /3C
- added copper zone on In2.Cu, net /3C
- added copper zone on In3.Cu, net /3C
- added copper zone on In4.Cu, net /3C
- added copper zone on B.Cu, net /4A
- added copper zone on F.Cu, net /4A
- added copper zone on In1.Cu, net /4A
- added copper zone on In2.Cu, net /4A
- added copper zone on In3.Cu, net /4A
- added copper zone on In4.Cu, net /4A
- added copper zone on B.Cu, net /4B
- added copper zone on F.Cu, net /4B
- added copper zone on In1.Cu, net /4B
- added copper zone on In2.Cu, net /4B
- added copper zone on In3.Cu, net /4B
- added copper zone on In4.Cu, net /4B
- added copper zone on B.Cu, net /4C
- added copper zone on F.Cu, net /4C
- added copper zone on In1.Cu, net /4C
- added copper zone on In2.Cu, net /4C
- added copper zone on In3.Cu, net /4C
- added copper zone on In4.Cu, net /4C
- added copper zone on B.Cu, net /CSA+
- added copper zone on In1.Cu, net /CSA+
- added copper zone on In2.Cu, net /CSA+
- added copper zone on In3.Cu, net /CSA+
- added copper zone on In4.Cu, net /CSA+
- added copper zone on B.Cu, net GND
- added copper zone on F.Cu, net GND
- added copper zone on In1.Cu, net GND
- added copper zone on In2.Cu, net GND
- added copper zone on In6.Cu, net GND
Other:
- copper layers 6 -> 8
