File: hardware/fc_pads.kicad_sch (KiCad schematic)
At the start: 41 parts, among them J15 5V, J16 5V, J17 5V, J18 5V, J19 5V, J20 5V, J21 5V, J22 5V, J23 5V, J24 5V, J25 5V, J26 5V, J27 5V, J28 5V, J29 5V, J30 5V, J31 5V, J32 5V, J33 5V, J34 5V, J35 5V, J37 5V, J38 5V, J39 5V, J40 5V, J41 5V, J42 5V, J43 5V, J44 5V, J45 5V, J46 5V, J47 5V, J48 5V, J49 5V, J50 5V, J51 5V, J52 5V, J53 5V, J54 5V, J55 5V, U12 SM06B-SRSS-TB(LF)(SN)

Commit message: Base: routing progress (~60%), netclass clearances relaxed
VBAT/Phase/Power/RF clearance lowered toward the 0.09 line standard; the
2 oz outer rule in the DRU still enforces 0.16 on F/B.Cu. Schematic sheets
resaved by eeschema, no circuit change.
Connections:
- net U1RX is gone; now on net UART1_RX: J46.1 (Pin_1), U12.6
Changed lines of the file:
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@@
+	(wire
+		(pts
+			(xy 55.88 113.03) (xy 55.88 107.95)
+		)
+		(stroke
+			(width 0)
+			(type default)
+		)
+	)
 	(wire
 		(pts
@@
 		(pts
 			(xy 78.74 62.23) (xy 78.74 64.77)
+		)
+		(stroke
+			(width 0)
+			(type default)
+		)
+	)
+	(wire
+		(pts
+			(xy 62.23 113.03) (xy 62.23 107.95)
 		)
 		(stroke
@@
 	(label "I2C0.SCL"
 		(at 77.47 146.05 90)
+		(effects
+			(font
+				(size 1.27 1.27)
+			)
+			(justify left bottom)
+		)
+	)
+	(label "U1RX"
+		(at 55.88 110.49 0)
 		(effects
 			(font
@@
 	(hierarchical_label "UART1_RX"
 		(shape input)
-		(at 55.88 107.95 270)
+		(at 55.88 113.03 270)
 		(effects
 			(font
@@
 	(hierarchical_label "UART1_TX"
 		(shape output)
-		(at 62.23 107.95 270)
-		(effects
-			(font
+		(at 62.23 113.03 270)
+		(effects
+			(font
