File: hardware/fc_pads.kicad_sch (KiCad schematic)
At the start: 37 parts, among them J15 5V, J16 5V, J17 5V, J18 5V, J19 5V, J20 5V, J21 5V, J22 5V, J24 5V, J25 5V, J27 5V, J28 5V, J29 5V, J31 5V, J32 5V, J33 5V, J35 5V, J37 5V, J38 5V, J39 5V, J40 5V, J41 5V, J42 5V, J43 5V, J44 5V, J45 5V, J46 5V, J47 5V, J48 5V, J49 5V, J50 5V, J51 5V, J52 5V, J53 5V, J54 5V, J55 5V, U12 SM06B-SRSS-TB(LF)(SN)

Commit message: chore: consolidate OpenAIO design assets and guidance
Parts:
- renumbered J21 to J10, J22 to J11, J54 to J12, J53 to J13, J52 to J14, J24 to J15, J25 to J16, J27 to J17, J28 to J18, J29 to J19, J31 to J20, J32 to J21, J33 to J22, J35 to J23, J37 to J24, J38 to J25, J39 to J26, J40 to J27, J41 to J28, J42 to J29, J15 to J3, J43 to J30, J44 to J31, J45 to J32, J46 to J33, J47 to J34, J48 to J35, J49 to J36, J50 to J37, J51 to J38, J16 to J4, J17 to J5, J18 to J6, J19 to J7, J55 to J8, J20 to J9, U12 to U10
