File: hardware/fc_pads.kicad_sch (KiCad schematic)
At the start: 41 parts, among them J15 5V, J16 5V, J17 5V, J18 5V, J19 5V, J20 5V, J21 5V, J22 5V, J23 5V, J24 5V, J25 5V, J26 5V, J27 5V, J28 5V, J29 5V, J30 5V, J31 5V, J32 5V, J33 5V, J34 5V, J35 5V, J37 5V, J38 5V, J39 5V, J40 5V, J41 5V, J42 5V, J43 5V, J44 5V, J45 5V, J46 5V, J47 5V, J48 5V, J49 5V, J50 5V, J51 5V, J52 5V, J53 5V, J54 5V, J55 5V, U12 SM06B-SRSS-TB(LF)(SN)

Commit message: Owner rules: no component silk, pad labels and values, no wordmark text, MPN + maker on every BOM line
The owner rules adopted in PLAN.md (pcb-agent-commons, 2026-10-06), applied
where they are local edits:

- No component silkscreen. J91's reference was the only visible one (Core
  B.Silkscreen, under the LGA) and is hidden. Footprint silk graphics removed
  per instance: Base 234, Core 72. Kept: connector outlines and pin-1 marks
  (USB1, U12 SH-6, Card1, JP1) and the LGA pin-1 marks (J90, J91). Base
  lib_footprint_mismatch warnings 31 -> 40 as a result.
- Solder-pad labels: Core J53 (GND) had none, now "gnd" in the style of J52's
  label. The SH-6 per-pin labels ("10v gnd T0", "R0 gnd R1") become the port
  name "DJI" (connectors: name and pin-1 mark only). Core J48-J51 have no room:
  0.5 mm to J44 above, 0.93 mm to the board edge below. CIRCUIT_REVIEW 8.3
  moves them off the LGA in R2, so their labels go with that move.
- Pad values: all 40 solder-pad symbols said "5V". Each now carries its
  function (5V, GND, LED, BUZ+/BUZ-, 10V, 4V5, CAM, VTX, SCL, SDA, TX0/RX0,
  TX1/RX1, PIO_TX0/PIO_RX0; off-board J19 ADC2, J22 GND, J46/J47 NC).
- No "Drone" text: the "OpenDrone" wordmark on Core F.Silkscreen (9 filled
  polygons in two groups) is removed; a TODO for the incutec wordmark from the
  brand repo sits on User.Comments (not fabricated). No other such text on any
  copper, mask or silk layer of either board.
- BOM: lines missing manufacturer or MPN 41 -> 1. MPNs come from
  PARTS-USED.md by LCSC number. Manufacturers come from the catalogue symbol,
  this design's spelling for the same MPN family, or the committed datasheet
  (NSIC, Sofng, Jiangsu Changjing, Hirose). Still open: Rsense2
  ASR-S-3-0.2F (C695806), whose manufacturer nothing in the catalogue states.
  U24 (board outline) and TP9 (BOOT solder pad) are not parts: excluded from
  BOM and position files.
- 0201 default / minimal capacitance: respected in the circuit commit (C26
  stays 0201; no belt-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
Parts:
- J17, J18, J22, J27, J28, J34, J35, J40, J43, J50, J53: value 5V -> GND
- J19: value 5V -> ADC2
- J20, J21, J31, J32: value 5V -> LED
- J23: value 5V -> SCL
- J26: value 5V -> SDA
- J29: value 5V -> BUZ-
- J33: value 5V -> BUZ+
- J38: value 5V -> CAM
- J39: value 5V -> VTX
- J41, J51: value 5V -> 10V
- J42, J52: value 5V -> 4V5
- J44: value 5V -> PIO_TX0
- J45: value 5V -> PIO_RX0
- J46, J47: value 5V -> NC
- J48: value 5V -> RX0
- J49: value 5V -> TX0
- J54: value 5V -> TX1
- J55: value 5V -> RX1
Changed lines of the file:
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@@
 			)
 		)
-		(property "Value" "5V"
+		(property "Value" "GND"
 			(at 50.546 53.848 90)
 			(hide yes)
@@
 			)
 		)
-		(property "Value" "5V"
+		(property "Value" "RX1"
 			(at 54.356 99.568 90)
 			(hide yes)
@@
 			)
 		)
-		(property "Value" "5V"
+		(property "Value" "SCL"
 			(at 78.994 154.432 90)
 			(hide yes)
@@
 			)
 		)
-		(property "Value" "5V"
+		(property "Value" "TX0"
 			(at 189.484 19.558 90)
 			(hide yes)
@@
 			)
 		)
-		(property "Value" "5V"
+		(property "Value" "GND"
 			(at 135.636 99.568 90)
 			(hide yes)
@@
 			)
 		)
-		(property "Value" "5V"
+		(property "Value" "VTX"
 			(at 132.334 99.568 90)
 			(hide yes)
@@
 			)
 		)
-		(property "Value" "5V"
+		(property "Value" "LED"
 			(at 56.896 53.848 90)
 			(hide yes)
@@
 			)
 		)
-		(property "Value" "5V"
+		(property "Value" "10V"
 			(at 199.644 19.558 90)
 			(hide yes)
@@
 			)
 		)
-		(property "Value" "5V"
+		(property "Value" "10V"
 			(at 141.986 99.568 90)
 			(hide yes)
@@
 			)
 		)
-		(property "Value" "5V"
+		(property "Value" "CAM"
 			(at 125.984 99.568 90)
 			(hide yes)
@@
 			)
 		)
-		(property "Value" "5V"
+		(property "Value" "GND"
 			(at 83.566 24.638 90)
 			(hide yes)
@@
 			)
 		)
-		(property "Value" "5V"
+		(property "Value" "GND"
 			(at 62.484 154.432 90)
 			(hide yes)
@@
 			)
 		)
-		(property "Value" "5V"
+		(property "Value" "NC"
 			(at 179.324 19.558 90)
 			(hide yes)
@@
 			)
 		)
-		(property "Value" "5V"
+		(property "Value" "LED"
 			(at 89.916 24.638 90)
 			(hide yes)
@@
 			)
 		)
-		(property "Value" "5V"
+		(property "Value" "GND"
 			(at 110.236 99.568 90)
 			(hide yes)
@@
 			)
 		)
-		(property "Value" "5V"
+		(property "Value" "GND"
 			(at 98.044 154.432 90)
 			(hide yes)
@@
 			)
 		)
-		(property "Value" "5V"
+		(property "Value" "GND"
 			(at 156.464 154.432 90)
 			(hide yes)
@@
 			)
 		)
-		(property "Value" "5V"
+		(property "Value" "BUZ+"
 			(at 93.726 99.568 90)
 			(hide yes)
@@
 			)
 		)
-		(property "Value" "5V"
+		(property "Value" "NC"
 			(at 174.244 19.558 90)
 			(hide yes)
@@
 			)
 		)
-		(property "Value" "5V"
+		(property "Value" "BUZ-"
 			(at 87.376 99.568 90)
 			(hide yes)
@@
 			)
 		)
-		(property "Value" "5V"
+		(property "Value" "LED"
 			(at 56.896 24.638 90)
 			(hide yes)
@@
 			)
 		)
-		(property "Value" "5V"
+		(property "Value" "ADC2"
 			(at 54.864 154.432 90)
 			(hide yes)
@@
 			)
 		)
-		(property "Value" "5V"
+		(property "Value" "GND"
 			(at 50.546 24.638 90)
 			(hide yes)
@@
 			)
 		)
-		(property "Value" "5V"
+		(property "Value" "4V5"
 			(at 150.114 154.432 90)
 			(hide yes)
@@
 			)
 		)
-		(property "Value" "5V"
+		(property "Value" "GND"
 			(at 194.564 19.558 90)
 			(hide yes)
@@
 			)
 		)
-		(property "Value" "5V"
+		(property "Value" "GND"
 			(at 67.056 99.568 90)
 			(hide yes)
@@
 			)
 		)
-		(property "Value" "5V"
+		(property "Value" "4V5"
 			(at 73.406 99.568 90)
 			(hide yes)
@@
 			)
 		)
-		(property "Value" "5V"
+		(property "Value" "TX1"
 			(at 60.706 99.568 90)
 			(hide yes)
@@
 			)
 		)
-		(property "Value" "5V"
+		(property "Value" "GND"
 			(at 83.566 53.848 90)
 			(hide yes)
@@
 			)
 		)
-		(property "Value" "5V"
+		(property "Value" "RX0"
 			(at 184.404 19.558 90)
 			(hide yes)
@@
 			)
 		)
-		(property "Value" "5V"
+		(property "Value" "PIO_TX0"
 			(at 162.814 154.432 90)
 			(hide yes)
@@
 			)
 		)
-		(property "Value" "5V"
+		(property "Value" "SDA"
 			(at 85.344 154.432 90)
 			(hide yes)
@@
 			)
 		)
-		(property "Value" "5V"
+		(property "Value" "PIO_RX0"
 			(at 169.164 154.432 90)
 			(hide yes)
@@
 			)
 		)
-		(property "Value" "5V"
+		(property "Value" "LED"
 			(at 89.916 53.848 90)
 			(hide yes)

Commit message: Schematic: LGA nets per the R2a spec, S1/S2/B2/D7
- LGA (core_interface, generated by tools/lga_gen.py --sheet and re-saved by
  kicad-cli): J90/J91 get the 46 pins and nets of LGA_SPEC.md. 10V_ENABLE
  (B1), +3.3V (S1) and +10V (S2) no longer cross; PU0RX, SWDIO, SWCLK do.
- B2: SH-6 U12 pin 6 (DJI SBUS) leaves UART1_RX (ESP32-C3 TX) and joins
  PU0RX (RP2354A GPIO3, PIO UART0 RX); PU0RX becomes a global net so it
  crosses the LGA.
- D7: RP2354A SWCLK/SWDIO (U2.24/.25, no-connect before) go to the LGA and
  to TP32 SWCLK / TP31 SWDIO, 0.8 mm test pads on the Base (not in the BOM).
- S2: VTX pads move to the Base next to the SH-6: J41 +10V and J51 (was a
  second +10V pad on the Core) GND, on lib:SolderPad_1.2x1.2mm.
- S1: U7 LP5912-3.3 and its caps move to the Core (board assignment is by
  footprint, see the board commit). CIN C26 becomes the 0402 1 uF 25 V
  CL05A105KA5NQNC (C52923) the spec places; the 0201 was the R1 stop-gap.
- D6/R24, the green power LED, was on +3.3V on the Base, which no longer
  exists there. Instead of moving it to the Core or deleting it (spec
  section 2), R24 now takes +3V3 (TLV75533 U23, fed from the same +4v5):
  same LED, same parts, no Core space used.

ERC: 31 errors before and after, same types (bus_to_net_conflict 3,
hier_label_mismatch 1, pin_not_connected 1, pin_not_driven 16, pin_to_pin 1,
power_pin_not_driven 9). Netlist J90/J91 checked pad by pad against
lga_spec.json: 0 mismatches.

Co-Authored-By: Claude Opus 5.5 <noreply@anthropic.com>
Claude-Session: https://claude.ai/code/session_01KTp3FLjVXfXdWrkmr6af7d
Parts:
- J41: footprint lib:small_pad -> lib:SolderPad_1.2x1.2mm
- J51: value 10V -> GND; footprint lib:small_pad -> lib:SolderPad_1.2x1.2mm
Connections:
- net +10V: no longer J51.1 (Pin_1)
- net GND: now also J51.1 (Pin_1)
- net UART1_RX: no longer J46.1 (Pin_1), U12.6
- net PIOUART0_RX renamed PU0RX
- net PU0RX: now also J46.1 (Pin_1), U12.6
Changed lines of the file:
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@@
 		)
 	)
-	(label "PU0RX"
-		(at 167.64 146.05 90)
+	(label "I2C0.SDA"
+		(at 83.82 146.05 90)
 		(effects
 			(font
@@
 		)
 	)
-	(label "I2C0.SDA"
-		(at 83.82 146.05 90)
+	(label "I2C0.SCL"
+		(at 77.47 146.05 90)
 		(effects
 			(font
@@
 	)
 	(label "U1RX"
-		(at 172.72 44.45 0)
+		(at 55.88 110.49 0)
 		(effects
 			(font
@@
 		)
 	)
-	(label "I2C0.SCL"
-		(at 77.47 146.05 90)
+	(global_label "PU0RX"
+		(shape bidirectional)
+		(at 172.72 44.45 0)
 		(effects
 			(font
 				(size 1.27 1.27)
 			)
-			(justify left bottom)
+			(justify left)
+		)
+		(property "Intersheetrefs" "${INTERSHEET_REFS}"
+			(at 172.72 44.45 0)
+			(hide yes)
+			(show_name no)
+			(do_not_autoplace no)
+			(effects
+				(font
+					(size 1.27 1.27)
+				)
+			)
 		)
 	)
-	(label "U1RX"
-		(at 55.88 110.49 0)
+	(global_label "PU0RX"
+		(shape bidirectional)
+		(at 167.64 146.05 90)
 		(effects
 			(font
 				(size 1.27 1.27)
 			)
-			(justify left bottom)
+			(justify left)
+		)
+		(property "Intersheetrefs" "${INTERSHEET_REFS}"
+			(at 167.64 146.05 0)
+			(hide yes)
+			(show_name no)
+			(do_not_autoplace no)
+			(effects
+				(font
+					(size 1.27 1.27)
+				)
+			)
 		)
 	)
@@
 			)
 		)
-		(property "Value" "10V"
+		(property "Value" "GND"
 			(at 199.644 19.558 90)
 			(hide yes)
@@
 			)
 		)
-		(property "Footprint" "lib:small_pad"
+		(property "Footprint" "lib:SolderPad_1.2x1.2mm"
 			(at 198.12 22.86 0)
 			(hide yes)
@@
 			)
 		)
-		(property "Footprint" "lib:small_pad"
+		(property "Footprint" "lib:SolderPad_1.2x1.2mm"
 			(at 143.51 102.87 0)
 			(hide yes)
@@
 	)
 	(symbol
-		(lib_id "power:+12V")
-		(at 191.77 31.75 180)
+		(lib_id "power:GND")
+		(at 191.77 31.75 0)
 		(unit 1)
 		(body_style 1)
@@
 		(dnp no)
 		(property "Reference" "#PWR0130"
-			(at 191.77 27.94 0)
+			(at 191.77 38.1 0)
 			(hide yes)
 			(show_name no)
@@
 			)
 		)
-		(property "Value" "+10V"
-			(at 191.77 37.846 90)
+		(property "Value" "GND"
+			(at 191.77 35.56 0)
 			(show_name no)
 			(do_not_autoplace no)
@@
 			)
 		)
-		(property "Description" "Power symbol creates a global label with name \"+12V\""
+		(property "Description" "Power symbol creates a global label with name \"GND\" , ground"
 			(at 191.77 31.75 0)
 			(hide yes)
