File: hardware/rx_esp32c3_sx1281.kicad_sch (KiCad schematic)
At the start: 43 parts, among them U21 SX1281IMLTRT, U22 ESP32-C3, U23 TLV75533PDQNR, X2 CJ17-400001010B20

Commit message: chore: consolidate OpenAIO design assets and guidance
Parts:
- renumbered C82 to C100, C83 to C101, C84 to C102, C85 to C103, C86 to C104, C87 to C105, C88 to C106, C89 to C107, C65 to C83, C66 to C84, C67 to C85, C68 to C86, C69 to C87, C70 to C88, C71 to C89, C72 to C90, C73 to C91, C74 to C92, C75 to C93, C76 to C94, C77 to C95, C78 to C96, C79 to C97, C80 to C98, C81 to C99, D9 to D6, FL1 to FL2, L6 to L10, L7 to L11, L4 to L8, L5 to L9, OSC1 to OSC2, R111 to R93, R112 to R94, R113 to R95, R114 to R96, TP9 to TP11, U21 to U19, U22 to U20, U23 to U21
