File: hardware/rx_esp32c3_sx1281.kicad_sch (KiCad schematic)
At the start: 43 parts, among them U21 SX1281IMLTRT, U22 ESP32-C3, U23 TLV75533PDQNR, X2 CJ17-400001010B20

Commit message: Circuit: B3 bulk caps and ESP32-C3FH4, LDO caps, BMI270 aux pins, BOOTSEL 1k, unused pads
CIRCUIT_REVIEW B3, S2, S4, S5 and decision D9; LAYOUT_REVIEW 5.3 (pure
clean-up). Values and parts from hardware/KiCad-Library/PARTS-USED.md.

- B3: the 16 +BATT bulk caps had value "C" and no part. C90-C103 (0805)
  4.7uF 50V X5R CL21A475KBQNNNE (C98192, already C18/C19); C105/C106 (1206)
  4.7uF 50V X7R TCC1206X7R475K500HT (C380366, OpenESC).
- D9/B3: U22 is ESP32-C3FH4 (C2858491, in-package flash), as its NC SPI pins
  require; its in-package-flash pads 19, 21-24 deleted per instance (20 was
  already gone). L4 MPN MLZ2012M150WT000 (TDK, SX1281 reference BOM, LCSC not
  in the catalogue); D9 MPN/manufacturer/LCSC from the catalogue.
- S2, LP5912 windows (CIN > 0.5 uF effective, COUT 0.7-10 uF): U7 COUT C28
  22uF -> 1uF CL05A105KA5NQNC; U6 COUT C27 22uF -> 4.7uF CL05A475MP5NRNC;
  U7 CIN C26 100nF -> 1uF GRM033R61A105ME44D in the existing 0201 (an 0402
  does not fit beside U7 without moving parts; ~0.5 uF effective at 4.6 V,
  so it is marginal until U7 moves to the Core in R2, decision S1).
- S4: BMI270 U8 ASDx/ASCx (pins 2/3) were on GND, which the datasheet
  forbids; now +3.3V (VDDIO), valid for the LSM6DSV16X option too.
  Schematic: the GND drop replaced by a +3.3V symbol. Core: pads 2/3 and the
  via between them re-netted, 0.15 mm In3 stub to the In3 +3.3V pour.
- S5: BOOTSEL resistor R7 10k -> 1k (0201WMF1001TEE, C270365): 10k with the
  32k minimum pull-up gave 0.79 V against VIL 0.8 V.
- LAYOUT_REVIEW 5.3, pads on no net with nothing attached: U13/U15/U17/U19
  (AT32F421) 3, 8, 9, 12, 23, 24, 26-28; U14/U16/U18/U20 (NSG2065Q) NC 5, 7,
  8, 21; U7 NC 2; U21 6 (XTB, TCXO), 9, 10 (DIO2/3); Core U2 55-59 (QSPI,
  in-package flash). 60 pads in all; U8 kept for joint symmetry. AT32
  firmware must keep the dropped pins as outputs or pulled.
- Footprint values and fields synced from the schematic for the changed refs.

Deferred: RX LED D9 to +4v5 (S10). +4v5 copper is 1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
Parts:
- D9: LCSC (none) -> C5349953; MPN (none) -> XL-1010RGBC-2812B; Manufacturer (none) -> XINGLIGHT
- L4: MPN (none) -> MLZ2012M150WT000; Manufacturer (none) -> TDK
- U22: value ESP32-C3 -> ESP32-C3FH4; LCSC (none) -> C2858491; MPN (none) -> ESP32-C3FH4; Manufacturer (none) -> Espressif Systems
Changed lines of the file:
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@@
 			)
 		)
+		(property "MPN" "MLZ2012M150WT000"
+			(at 97.536 85.09 90)
+			(hide yes)
+			(show_name no)
+			(do_not_autoplace no)
+			(effects
+				(font
+					(size 1.27 1.27)
+				)
+			)
+		)
+		(property "Manufacturer" "TDK"
+			(at 97.536 85.09 90)
+			(hide yes)
+			(show_name no)
+			(do_not_autoplace no)
+			(effects
+				(font
+					(size 1.27 1.27)
+				)
+			)
+		)
 		(pin "2"
 		)
@@
 			)
 		)
+		(property "MPN" "XL-1010RGBC-2812B"
+			(at 129.54 184.0798 0)
+			(hide yes)
+			(show_name no)
+			(do_not_autoplace no)
+			(effects
+				(font
+					(size 1.27 1.27)
+				)
+			)
+		)
+		(property "Manufacturer" "XINGLIGHT"
+			(at 129.54 184.0798 0)
+			(hide yes)
+			(show_name no)
+			(do_not_autoplace no)
+			(effects
+				(font
+					(size 1.27 1.27)
+				)
+			)
+		)
+		(property "LCSC" "C5349953"
+			(at 129.54 184.0798 0)
+			(hide yes)
+			(show_name no)
+			(do_not_autoplace no)
+			(effects
+				(font
+					(size 1.27 1.27)
+				)
+			)
+		)
 		(pin "1"
 		)
@@
 			)
 		)
-		(property "Value" "ESP32-C3"
+		(property "Value" "ESP32-C3FH4"
 			(at 224.3933 248.92 0)
 			(show_name no)
@@
 			)
 		)
-		(property "Datasheet" "https://www.espressif.com/sites/default/files/documentation/esp32-c3_datasheet_en.pdf"
+		(property "Datasheet" "${OPENDRONE_LIB}/datasheet/ESP32-C3FH4.pdf"
 			(at 222.758 220.98 0)
 			(hide yes)
@@
 			)
 		)
+		(property "MPN" "ESP32-C3FH4"
+			(at 224.3933 248.92 0)
+			(hide yes)
+			(show_name no)
+			(do_not_autoplace no)
+			(effects
+				(font
+					(size 1.27 1.27)
+				)
+				(justify left)
+			)
+		)
+		(property "Manufacturer" "Espressif Systems"
+			(at 224.3933 248.92 0)
+			(hide yes)
+			(show_name no)
+			(do_not_autoplace no)
+			(effects
+				(font
+					(size 1.27 1.27)
+				)
+				(justify left)
+			)
+		)
+		(property "LCSC" "C2858491"
+			(at 224.3933 248.92 0)
+			(hide yes)
+			(show_name no)
+			(do_not_autoplace no)
+			(effects
+				(font
+					(size 1.27 1.27)
+				)
+				(justify left)
+			)
+		)

Commit message: Owner rules: no component silk, pad labels and values, no wordmark text, MPN + maker on every BOM line
The owner rules adopted in PLAN.md (pcb-agent-commons, 2026-10-06), applied
where they are local edits:

- No component silkscreen. J91's reference was the only visible one (Core
  B.Silkscreen, under the LGA) and is hidden. Footprint silk graphics removed
  per instance: Base 234, Core 72. Kept: connector outlines and pin-1 marks
  (USB1, U12 SH-6, Card1, JP1) and the LGA pin-1 marks (J90, J91). Base
  lib_footprint_mismatch warnings 31 -> 40 as a result.
- Solder-pad labels: Core J53 (GND) had none, now "gnd" in the style of J52's
  label. The SH-6 per-pin labels ("10v gnd T0", "R0 gnd R1") become the port
  name "DJI" (connectors: name and pin-1 mark only). Core J48-J51 have no room:
  0.5 mm to J44 above, 0.93 mm to the board edge below. CIRCUIT_REVIEW 8.3
  moves them off the LGA in R2, so their labels go with that move.
- Pad values: all 40 solder-pad symbols said "5V". Each now carries its
  function (5V, GND, LED, BUZ+/BUZ-, 10V, 4V5, CAM, VTX, SCL, SDA, TX0/RX0,
  TX1/RX1, PIO_TX0/PIO_RX0; off-board J19 ADC2, J22 GND, J46/J47 NC).
- No "Drone" text: the "OpenDrone" wordmark on Core F.Silkscreen (9 filled
  polygons in two groups) is removed; a TODO for the incutec wordmark from the
  brand repo sits on User.Comments (not fabricated). No other such text on any
  copper, mask or silk layer of either board.
- BOM: lines missing manufacturer or MPN 41 -> 1. MPNs come from
  PARTS-USED.md by LCSC number. Manufacturers come from the catalogue symbol,
  this design's spelling for the same MPN family, or the committed datasheet
  (NSIC, Sofng, Jiangsu Changjing, Hirose). Still open: Rsense2
  ASR-S-3-0.2F (C695806), whose manufacturer nothing in the catalogue states.
  U24 (board outline) and TP9 (BOOT solder pad) are not parts: excluded from
  BOM and position files.
- 0201 default / minimal capacitance: respected in the circuit commit (C26
  stays 0201; no belt-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
Parts:
- AE2: MPN (none) -> 2450AT18A100E; Manufacturer (none) -> JOHANSON(约翰逊)
- C65, C66, C70, C71, C76, C78, C79: MPN (none) -> GRM033R61E104KE14D; Manufacturer (none) -> Murata Electronics
- C67, C73, C80: MPN (none) -> GRM033R61A103KA01J; Manufacturer (none) -> Murata Electronics
- C68: MPN (none) -> GRM033R60J474KE90D; Manufacturer (none) -> Murata Electronics
- C69: MPN (none) -> 0201B102K500NT; Manufacturer (none) -> FH (Guangdong Fenghua)
- C72, C74: MPN (none) -> GRM0335C1H150JA01D; Manufacturer (none) -> Murata Electronics
- C75: MPN (none) -> GRM155R60J106ME44D; Manufacturer (none) -> Murata Electronics
- C77, C81, C83, C84, C85, C86: MPN (none) -> GRM033R61A105ME44D; Manufacturer (none) -> Murata Electronics
- C82, C88: MPN (none) -> CL05A106MQ5NUNC; Manufacturer (none) -> Samsung Electro-Mechanics
- C87, C89: MPN (none) -> GRM0335C1H1R2BA01D; Manufacturer (none) -> Murata Electronics
- JP1: MPN (none) -> U.FL-R-SMT-1(80); Manufacturer (none) -> Hirose
- L5: MPN (none) -> LQP03TN24NH02D; Manufacturer (none) -> Murata Electronics
- L6: MPN (none) -> LQP03TN2N0B02D; Manufacturer (none) -> Murata Electronics
- L7: MPN (none) -> LQP03TN2N5C02D; Manufacturer (none) -> Murata Electronics
- OSC1: MPN (none) -> OW7EL89CENUNFAYLC-52M; Manufacturer (none) -> TXC
- R111, R112, R113, R114: MPN (none) -> RC0201FR-0710KL; Manufacturer (none) -> YAGEO
- TP9: now left out of the parts list
- U21: MPN (none) -> SX1281IMLTRT; Manufacturer (none) -> Semtech
- U23: MPN (none) -> TLV75533PDQNR; Manufacturer (none) -> Texas Instruments
- X2: MPN (none) -> CJ17-400001010B20; Manufacturer (none) -> Jiangsu Changjing Electronics
