File: hardware/core_interface.kicad_sch (KiCad schematic)
At the start: 2 parts, among them J90 Core_LGA, J91 Core_LGA

Commit message: DFM: Core PCBA as a consigned BOM/CPL line on the Base, panel plan, order notes (DFM-09, DFM-10)
DFM-09: J90 now stands for the assembled Core on the Base BOM and position
files. Schematic (core_interface.kicad_sch, J90 only, via kicad-skip and
kicad-cli sch upgrade): in_bom and in_pos_files yes, Value "OpenAIO-Core PCBA
(consigned)", hidden fields Manufacturer "OpenDrone", MPN "OpenAIO-Core
PCBA" and "BOM note" with the pick-point: the CPL point is the J90 origin
(80.25, 61.65, top, 0 deg); pick on U2 (flat 7 x 7 mm QFN top) at -3.77,
+2.25 mm from it; the Core outline centre is at -1.03, +0.23 mm. The board
footprint carries the same value and fields, and is no longer excluded from
BOM/pos. lga_gen.py and lib Core_LGA_land write (attr smd) for the land; J91
on the Core stays excluded. ERC 31 errors (unchanged); parity unchanged.

DFM-10: research/review-2026-10/PANEL.md proposes the panels without
changing either outline. Measured free edge runs (nothing within 0.5 mm):
Core 21.6 mm total, longest 11.1 mm on the bottom edge; Base 9.4 mm, longest
2.9 mm at x = 91.9. No 5 mm tab can keep parts 3 mm away. Proposal: Core
3 x 2 (72.2 x 51.8 mm) and Base 2 x 2 (52.6 x 62.6 mm), 5 mm rails with three
1 mm fiducials on F and B and four tooling holes, solid 1.5-3.0 mm tabs only
on the free runs, router depanel (flush, no nubs next to U12/Q13/Q11),
2.5 mm gap at USB1.

NEXTPCB.md: questions 12-14 (0.5 mm fiducials, Core flatness and 0.12 mm
Base top stencil, narrow router-cut tabs) and section 4.7 "Order notes":
stencils per side, LGA joint volume and the <= 0.10 mm Core bow/twist
requirement, LGA copper clearances, mask, fiducials, panels.

Co-Authored-By: Claude Opus 5.5 <noreply@anthropic.com>
Claude-Session: https://claude.ai/code/session_01KTp3FLjVXfXdWrkmr6af7d
Parts:
- J90: value Core_LGA -> OpenAIO-Core PCBA (consigned); BOM note (none) -> Consigned (C): the assembled Core from the Core order. CPL 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; MPN (none) -> OpenAIO-Core PCBA; Manufacturer (none) -> OpenDrone; now in the parts list
Changed lines of the file:
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@@
 		(body_style 1)
 		(exclude_from_sim no)
-		(in_bom no)
+		(in_bom yes)
 		(on_board yes)
-		(in_pos_files no)
+		(in_pos_files yes)
 		(dnp no)
 		(fields_autoplaced yes)
@@
 			)
 		)
-		(property "Value" "Core_LGA"
+		(property "Value" "OpenAIO-Core PCBA (consigned)"
 			(at 77.47 44.45 0)
 			(show_name no)
@@
 			(at 77.47 105.41 0)
 			(hide yes)
+			(show_name no)
+			(do_not_autoplace no)
+			(effects
+				(font
+					(size 1.27 1.27)
+				)
+				(justify left)
+			)
+		)
+		(property "Manufacturer" "OpenDrone"
+			(at 77.47 105.41 0)
+			(hide yes)
+			(show_name no)
+			(do_not_autoplace no)
+			(effects
+				(font
+					(size 1.27 1.27)
+				)
+				(justify left)
+			)
+		)
+		(property "MPN" "OpenAIO-Core PCBA"
+			(at 77.47 105.41 0)
+			(hide yes)
+			(show_name no)
+			(do_not_autoplace no)
+			(effects
+				(font
+					(size 1.27 1.27)
+				)
+				(justify left)
+			)
+		)
+		(property "BOM note" "Consigned (C): the assembled Core from the Core order. CPL point = J90 origin (LGA pattern centre), top, 0 deg. Pick on U2 (RP2354A, flat 7x7 mm top) at -3.77, +2.25 mm from the CPL point; Core outline centre at -1.03, +0.23 mm."
+			(at 77.47 105.41 0)
+			(hide yes)
