File: hardware/fc_rp2350a.kicad_sch (KiCad schematic)
At the start: 49 parts, among them Q1 AP1606, Q2 AP1606, U1 TS2306A 240GF MSM 9_C2976675, U2 RP2354A, X1 XTM25012000JT00351001

Commit message: ELRS_EN on GPIO27, SWD test pads TP42/TP43
- GPIO27 (U2.41) -> ESP32-C3 CHIP_EN (net ELRS_EN; R114 keeps ELRS on).
  Betaflight PINIO1 (inverted push-pull) holds ELRS in reset on demand, so
  the DJI SBUS on SH-6 pin 6 can own UART1_RX.
- SWCLK (U2.24) -> TP42, SWDIO (U2.25) -> TP43, D1.0 pads, parked right of
  the outline for placement.
- tools/sch_debug_pins.py (sexpdata); netlist diff: only these nets change.
- Board synced: 0 DRC errors, unconnected 70 -> 72 (ELRS_EN, SWDIO).
  U2 pad 24 (SWCLK) is still missing: pad 23 (+1.1V) cannot escape past XOUT/C4
  and the +3.3V via under it; needs a hand rework of the crystal corner.

Co-Authored-By: Claude Opus 5.5 <noreply@anthropic.com>
Parts:
- added TP42, TP43: TestPoint, lib:TestPoint_Pad_D1.0mm, symbol lib:TestPoint
Connections:
- net SWCLK: now reaches U2.24 (SWCLK)
- net SWCLK: now also TP42.1
- net SWDIO: now reaches U2.25 (SWDIO)
- net SWDIO: now also TP43.1
- net ELRS_EN: now reaches U2.41 (GPIO27_ADC1)
- no-connect marks 10 -> 7
Changed lines of the file:
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@@
 	)
 	(no_connect
-		(at 321.31 250.19)
-	)
-	(no_connect
-		(at 270.51 196.85)
-	)
-	(no_connect
 		(at 270.51 217.17)
 	)
@@
 	)
 	(no_connect
-		(at 270.51 199.39)
-	)
-	(no_connect
 		(at 270.51 209.55)
 	)
@@
 		)
 	)
+	(label "SWCLK"
+		(at 270.51 196.85 180)
+		(effects
+			(font
+				(size 1.27 1.27)
+			)
+			(justify right)
+		)
+	)
 	(label "XIN"
 		(at 270.51 179.07 180)
@@
 		)
 	)
+	(label "SWDIO"
+		(at 270.51 199.39 180)
+		(effects
+			(font
+				(size 1.27 1.27)
+			)
+			(justify right)
+		)
+	)
 	(global_label "USB_D-"
 		(shape bidirectional)
@@
 		)
 	)
+	(global_label "ELRS_EN"
+		(shape bidirectional)
+		(at 321.31 250.19 0)
+		(effects
+			(font
+				(size 1.27 1.27)
+			)
+			(justify left)
+		)
+		(property "Intersheetrefs" "${INTERSHEET_REFS}"
+			(at 321.31 250.19 0)
+			(hide yes)
+			(show_name no)
+			(do_not_autoplace no)
+			(effects
+				(font
+					(size 1.27 1.27)
+				)
+			)
+		)
+	)
 	(global_label "USB_D+"
 		(shape bidirectional)
@@
 	)
 	(symbol
+		(lib_id "lib:TestPoint")
+		(at 270.51 196.85 90)
+		(unit 1)
+		(body_style 1)
+		(exclude_from_sim no)
+		(in_bom no)
+		(on_board yes)
+		(in_pos_files yes)
+		(dnp no)
+		(fields_autoplaced yes)
+		(property "Reference" "TP42"
+			(at 266.415 192.2779 0)
+			(show_name no)
+			(do_not_autoplace no)
+			(effects
+				(font
+					(size 1.27 1.27)
+				)
+				(justify left)
+			)
+		)
+		(property "Value" "TestPoint"
+			(at 266.415 194.8179 0)
+			(show_name no)
+			(do_not_autoplace no)
+			(effects
+				(font
+					(size 1.27 1.27)
+				)
+				(justify left)
+			)
+		)
+		(property "Footprint" "lib:TestPoint_Pad_D1.0mm"
+			(at 269.59 196.85 0)
+			(hide yes)
+			(show_name no)
+			(do_not_autoplace no)
+			(effects
+				(font
+					(size 1.27 1.27)
+				)
+			)
+		)
+		(property "Datasheet" ""
+			(at 269.59 196.85 0)
+			(hide yes)
+			(show_name no)
+			(do_not_autoplace no)
+			(effects
+				(font
+					(size 1.27 1.27)
+				)
+			)
+		)
+		(property "Description" "test point"
+			(at 264.51 196.85 0)
+			(hide yes)
+			(show_name no)
+			(do_not_autoplace no)
+			(effects
+				(font
+					(size 1.27 1.27)
+				)
+			)
+		)
+		(pin "1"
+		)
+		(instances
+			(project "OpenAIO"
+				(path "/fb88b6f9-ee39-4640-a9d4-04a17ceeac64/01bcb197-c5fe-4dbd-addf-fd4e1bc6a2d2"
+					(reference "TP42")
+					(unit 1)
+				)
+			)
+		)
+	)
+	(symbol
 		(lib_id "lib:GND")
 		(at 110.49 200.66 0)
@@
 					(unit 1)
 				)
+			)
+		)
+	)
+	(symbol
+		(lib_id "lib:TestPoint")
+		(at 270.51 199.39 90)
+		(unit 1)
+		(body_style 1)
+		(exclude_from_sim no)
+		(in_bom no)
+		(on_board yes)
+		(in_pos_files yes)
+		(dnp no)
+		(fields_autoplaced yes)
+		(property "Reference" "TP43"
+			(at 266.415 194.8179 0)
+			(show_name no)
+			(do_not_autoplace no)
+			(effects
+				(font
+					(size 1.27 1.27)
+				)
+				(justify left)
+			)
+		)
+		(property "Value" "TestPoint"
+			(at 266.415 197.3579 0)
+			(show_name no)
+			(do_not_autoplace no)
+			(effects
+				(font
+					(size 1.27 1.27)
+				)
+				(justify left)
+			)
+		)
+		(property "Footprint" "lib:TestPoint_Pad_D1.0mm"
+			(at 269.59 199.39 0)
+			(hide yes)
+			(show_name no)
+			(do_not_autoplace no)
+			(effects
+				(font
+					(size 1.27 1.27)
+				)
+			)
+		)
+		(property "Datasheet" ""
+			(at 269.59 199.39 0)
+			(hide yes)
+			(show_name no)
+			(do_not_autoplace no)
+			(effects
+				(font
+					(size 1.27 1.27)
+				)
+			)
+		)
+		(property "Description" "test point"
+			(at 264.51 199.39 0)
+			(hide yes)
+			(show_name no)
+			(do_not_autoplace no)
+			(effects
+				(font
+					(size 1.27 1.27)
+				)
+			)
+		)
+		(pin "1"
+		)
+		(instances
+			(project "OpenAIO"
+				(path "/fb88b6f9-ee39-4640-a9d4-04a17ceeac64/01bcb197-c5fe-4dbd-addf-fd4e1bc6a2d2"
+					(reference "TP43")
+					(unit 1)
+				)

Commit message: Owner: routing in progress
Co-Authored-By: Claude Opus 5.5 <noreply@anthropic.com>
Parts:
- removed TP42, TP43: TestPoint, lib:TestPoint_Pad_D1.0mm, symbol lib:TestPoint
Connections:
- net SWCLK: no longer names the net of U2.24 (SWCLK)
- net SWDIO: no longer names the net of U2.25 (SWDIO)
- no-connect marks 7 -> 9
Other:
- moved on the sheet: R8, TP24, TP25
